File: schematics/kicad/sun2_mmu.kicad_sch (KiCad schematic)
At the start: 23 parts, among them U1 74F08, U300 LS2518, U301 LS2518, U302 74F257, U303 2168, U304 2168, U305 2168, U306 2168, U307 2168, U308 2168, U309 2168, U310 2168, U314 2949, U315 74F151, U316 P16R4, U317 2949, U318 2949, U319 2949, U320 2949, U321 74LS138, U322 74LS138, U323 74LS138, U324 74LS138

Commit message: Finish MMU
Parts:
- added S300: 4.7 KOhm, Resistor_THT:R_Array_SIP10, symbol Device:R_Network09_US
Connections:
- net ACC: now also U316.14 (Q3), U316.18 (O1), U317.6 (A5)
- net CXS0: now also U301.2 (Q0)
- net CXS1: now also U301.5 (Q1)
- net CXS2: now also U301.11 (Q2)
- net CXS3: now also U301.14 (Q3)
- net GND: now also U300.8 (GND), U301.8 (GND), U314.10 (GND), U315.1 (D3), U315.12 (D7), U315.8 (GND), U316.10 (GND), U317.10 (GND), U318.10 (GND), U319.10 (GND), U320.10 (GND), U321.5 (E2), S300.1 (common)
- net IA16: now also U314.1 (A0)
- net IA17: now also U314.2 (A1)
- net IA18: now also U314.3 (A2)
- net IA19: now also U314.4 (A3)
- net IA20: now also U314.5 (A4)
- net IA21: now also U314.6 (A5)
- net IA22: now also U314.7 (A6)
- net IA23: now also U314.8 (A7)
- net MA11: now also U319.1 (A0)
- net MA12: now also U319.2 (A1)
- net MA13: now also U319.3 (A2)
- net MA14: now also U319.4 (A3)
- net MA15: now also U319.5 (A4)
- net MA16: now also U319.6 (A5)
- net MA17: now also U319.7 (A6)
- net MA18: now also U319.8 (A7)
- net MA19: now also U320.1 (A0)
- net MA20: now also U320.2 (A1)
- net MA21: now also U320.3 (A2)
- net MA22: now also U320.4 (A3)
- net MOD: now also U316.15 (Q2), U316.4 (D2), U317.5 (A4)
- net P.FC2: now also U315.9 (C), U316.8 (D6), U321.3 (A2)
- net PROT0: now also U315.2 (D2), U318.2 (A1)
- net PROT1: now also U315.3 (D1), U318.3 (A2)
- net PROT2: now also U315.4 (D0), U318.4 (A3)
- net PROT3: now also U315.13 (D6), U318.5 (A4)
- net PROT4: now also U315.14 (D5), U318.6 (A5)
- net PROT5: now also U315.15 (D4), U318.7 (A6)
- net TYPE0: now also U316.16 (Q1), U316.3 (D1), U317.7 (A6)
- net TYPE1: now also U316.17 (Q0), U316.2 (D0), U317.8 (A7)
- net TYPE2: now also U318.1 (A0)
- net VALID: now also U318.8 (A7)
- net VCC: now also U300.16 (VCC), U301.16 (VCC), U314.20 (VCC), U315.16 (VCC), U316.20 (VCC), U317.20 (VCC), U318.20 (VCC), U319.20 (VCC), U320.20 (VCC)
- net WR.PMAP0U\: now also U318.11 (R), U323.11 (O4)
- net WR.PMAP0X\: now also U1.3
- net WR.PMAP1L\: now also U319.11 (R), U322.10 (O5)
- net WR.PMAP1U\: now also U320.11 (R), U323.10 (O5)
- net WR.SMAP\: now also U314.11 (R), U322.9 (O6)
- net P.D7: now reaches U314.12 (B7)
- net P.D7: now also U317.12 (B7), U319.12 (B7)
- net P.D6: now reaches U314.13 (B6)
- net P.D6: now also U317.13 (B6), U319.13 (B6)
- net P.D5: now reaches U314.14 (B5)
- net P.D5: now also U317.14 (B5), U319.14 (B5)
- net P.D4: now reaches U314.15 (B4)
- net P.D4: now also U317.15 (B4), U319.15 (B4)
- net P.D3: now reaches U314.16 (B3)
- net P.D3: now also U300.13 (Y3), U300.15 (D3), U317.16 (B3), U319.16 (B3)
- net P.D2: now reaches U314.17 (B2)
- net P.D2: now also U300.10 (Y2), U300.12 (D2), U317.17 (B2), U319.17 (B2)
- net P.D1: now reaches U314.18 (B1)
- net P.D1: now also U300.4 (D1), U300.6 (Y1), U317.18 (B1), U319.18 (B1)
- net P.D0: now reaches U314.19 (B0)
- net P.D0: now also U300.1 (D0), U300.3 (Y0), U317.19 (B0), U319.19 (B0)
- net RD.SMAP\: now reaches U314.9 (T)
- net RD.SMAP\: now also U322.13 (O2)
- net P.D15: now reaches U320.12 (B7)
- net P.D15: now also U318.12 (B7)
- net P.D14: now reaches U320.13 (B6)
- net P.D14: now also U318.13 (B6)
- net P.D13: now reaches U320.14 (B5)
- net P.D13: now also U318.14 (B5)
- net P.D12: now reaches U320.15 (B4)
- net P.D12: now also U318.15 (B4)
- net P.D11: now reaches U320.16 (B3)
- net P.D11: now also U301.13 (Y3), U301.15 (D3), U318.16 (B3)
- net P.D10: now reaches U320.17 (B2)
- net P.D10: now also U301.10 (Y2), U301.12 (D2), U318.17 (B2)
- net P.D9: now reaches U320.18 (B1)
- net P.D9: now also U301.4 (D1), U301.6 (Y1), U318.18 (B1)
- net P.D8: now reaches U320.19 (B0)
- net P.D8: now also U301.1 (D0), U301.3 (Y0), U318.19 (B0)
- net Z0: now reaches U320.5 (A4)
- net Z0: now also S300.2 (R1)
- net Z1: now reaches U320.6 (A5)
- net Z1: now also S300.3 (R2)
- net Z2: now reaches U320.7 (A6)
- net Z2: now also S300.4 (R3)
- net Z3: now reaches U320.8 (A7)
- net Z3: now also S300.5 (R4)
- net RD.PMAP1U\: now reaches U320.9 (T)
- net RD.PMAP1U\: now also U323.14 (O1)
- net P.A1: now reaches U323.1 (A0)
- net P.A1: now also U322.1 (A0), U324.1 (A0)
- net RD.CXU\: now reaches U323.12 (O3)
- net RD.CXU\: now also U301.7 (OE)
- net RD.PMAP0U\: now reaches U323.15 (O0)
- net RD.PMAP0U\: now also U318.9 (T)
- net P.A2: now reaches U323.2 (A1)
- net P.A2: now also U322.2 (A1), U324.2 (A1)
- net R\/W: now reaches U323.3 (A2)
- net R\/W: now also U315.11 (A), U322.3 (A2), U324.3 (A2)
- net P.A3: now reaches U323.4 (E1)
- net P.A3: now also U322.4 (E1), U324.6 (E3)
- net P.MMU\: now reaches U323.5 (E2)
- net P.MMU\: now also U321.12 (O3), U322.5 (E2), U324.5 (E2)
- net UDS: now reaches U323.6 (E3)
- net WR.CXU\: now reaches U323.7 (O7)
- net WR.CXU\: now also U301.9 (CK)
- net Z4: now reaches U317.1 (A0)
- net Z4: now also S300.6 (R5)
- net WR.PMAP0L\: now reaches U317.11 (R)
- net WR.PMAP0L\: now also U1.2, U322.11 (O4)
- net Z5: now reaches U317.2 (A1)
- net Z5: now also S300.7 (R6)
- net Z6: now reaches U317.3 (A2)
- net Z6: now also S300.8 (R7)
- net Z7: now reaches U317.4 (A3)
- net Z7: now also S300.9 (R8)
- net RD.PMAP0L\: now reaches U317.9 (T)
- net RD.PMAP0L\: now also U322.15 (O0)
- net RD.CXL\: now reaches U322.12 (O3)
- net RD.CXL\: now also U300.7 (OE)
- net RD.PMAP1L\: now reaches U322.14 (O1)
- net RD.PMAP1L\: now also U319.9 (T)
- net LDS: now reaches U322.6 (E3)
- net WR.CXL\: now reaches U322.7 (O7)
- net WR.CXL\: now also U300.9 (CK)
- net P.FC0: now reaches U321.1 (A0)
- net P.FC1: now reaches U321.2 (A1)
- net P.FC1: now also U315.10 (B), U316.7 (D5)
- net P.AS\: now reaches U321.4 (E1)
- net P.BACK\: now reaches U321.6 (E3)
- net P.INTA\: now reaches U321.7 (O7)
- net P.SPROG\: now reaches U321.9 (O6)
- net C.S4\: now reaches U315.7 (S)
- net C.S6\: now reaches U1.1
- net C.S6\: now also U316.11 (OE)
- net C.S5: now reaches U316.1 (CLK)
- net C.S5: now also U316.12 (O3)
- net DIS\: now reaches U316.19 (O0)
- net ERR\: now reaches U316.5 (D3)
- net P.R/W\: now reaches U316.6 (D4)
- net BOOTEN\: now reaches U316.9 (D7)
- net WR.DIAG\: now reaches U324.10 (O5)
- net ED.ENABLE\: now reaches U324.12 (O3)
- net RD.ERROR\: now reaches U324.13 (O2)
- net RD.IDPROM\: now reaches U324.15 (O0)
- net DS\: now reaches U324.4 (E1)
- net WR.ENABLE\: now reaches U324.7 (O7)
- no-connect marks 0 -> 8
Other:
- note added: "CONTEXT REGISTER"
- note added: "PAGE MAP"
- note added: "PROTECTION DECODER"
- note added: "SEGMENT MAP"
- note added: "STATISTICS BIT LOGIC"
- note added: "TODO"
- moved on the sheet: U1A, U300, U301, U302, U303, U304, U305, U306, U307, U308, U309, U310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

Commit message: PROM, RTC, Registers work
Parts:
- renumbered U1 to U313
Connections:
- net ED.ENABLE\ renamed RD.ENABLE\
Changed lines of the file:
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@@
 		)
 	)
-	(hierarchical_label "ED.ENABLE\\"
-		(shape input)
+	(hierarchical_label "RD.ENABLE\\"
+		(shape output)
 		(at 50.8 177.8 0)
 		(effects
@@
 	)
 	(hierarchical_label "RD.IDPROM\\"
-		(shape input)
+		(shape output)
 		(at 50.8 170.18 0)
 		(effects
@@
 	)
 	(hierarchical_label "WR.ENABLE\\"
-		(shape input)
+		(shape output)
 		(at 50.8 187.96 0)
 		(effects
@@
 	)
 	(hierarchical_label "RD.ERROR\\"
-		(shape input)
+		(shape output)
 		(at 50.8 175.26 0)
 		(effects
@@
 	)
 	(hierarchical_label "WR.DIAG\\"
-		(shape input)
+		(shape output)
 		(at 50.8 182.88 0)
 		(effects
@@
 		(on_board yes)
 		(dnp no)
-		(property "Reference" "U1"
+		(property "Reference" "U313"
 			(at 177.546 189.23 0)
 			(effects
@@
 			(project "sun2"
 				(path "/67ee2072-0b57-4a50-8537-b17b5f651e89/ecd7f6d8-851f-4bf4-a445-bd7a2a0bfdc8"
-					(reference "U1")
+					(reference "U313")
 					(unit 1)
 				)
