File: schematics/kicad/sun2_mmu.kicad_sch (KiCad schematic)
At the start: 24 parts, among them U300 LS2518, U301 LS2518, U302 74F257, U303 2168, U304 2168, U305 2168, U306 2168, U307 2168, U308 2168, U309 2168, U310 2168, U313 74F08, U314 2949, U315 74F151, U316 P16R4, U317 2949, U318 2949, U319 2949, U320 2949, U321 74LS138, U322 74LS138, U323 74LS138, U324 74LS138

Commit message: Rasterop, parity, P2 work
Connections:
- net IA16: now also U305.2 (A5), U306.2 (A5), U307.2 (A5), U308.2 (A5), U309.2 (A5), U310.2 (A5)
- net IA17: now also U305.3 (A6), U306.3 (A6), U307.3 (A6), U308.3 (A6), U309.3 (A6), U310.3 (A6)
- net IA18: now also U305.4 (A7), U306.4 (A7), U307.4 (A7), U308.4 (A7), U309.4 (A7), U310.4 (A7)
- net IA19: now also U305.5 (A8), U306.5 (A8), U307.5 (A8), U308.5 (A8), U309.5 (A8), U310.5 (A8)
- net IA20: now also U305.6 (A9), U306.6 (A9), U307.6 (A9), U308.6 (A9), U309.6 (A9), U310.6 (A9)
- net IA21: now also U305.7 (A10), U306.7 (A10), U307.7 (A10), U308.7 (A10), U309.7 (A10), U310.7 (A10)
- net IA22: now also U305.8 (A11), U306.8 (A11), U307.8 (A11), U308.8 (A11), U309.8 (A11), U310.8 (A11)
- net IA23: now also U305.1 (A4), U306.1 (A4), U307.1 (A4), U308.1 (A4), U309.1 (A4), U310.1 (A4)
Changed lines of the file:
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@@
+		)
+	)
+	(label "IA19"
+		(at 207.01 44.45 180)
+		(effects
+			(font
+				(size 1.27 1.27)
+			)
+			(justify right bottom)
 		)
 	)
@@
 		)
 	)
+	(label "IA21"
+		(at 207.01 49.53 180)
+		(effects
+			(font
+				(size 1.27 1.27)
+			)
+			(justify right bottom)
+		)
+	)
 	(label "P.D6"
 		(at 321.31 113.03 0)
@@
 		)
 	)
+	(label "IA20"
+		(at 207.01 46.99 180)
+		(effects
+			(font
+				(size 1.27 1.27)
+			)
+			(justify right bottom)
+		)
+	)
 	(label "P.D12"
 		(at 321.31 149.86 0)
@@
 		)
 	)
+	(label "IA22"
+		(at 207.01 52.07 180)
+		(effects
+			(font
+				(size 1.27 1.27)
+			)
+			(justify right bottom)
+		)
+	)
 	(label "P.A1"
 		(at 19.05 170.18 0)
@@
 		)
 	)
+	(label "IA23"
+		(at 207.01 34.29 180)
+		(effects
+			(font
+				(size 1.27 1.27)
+			)
+			(justify right bottom)
+		)
+	)
 	(label "CXS3"
 		(at 102.87 91.44 0)
@@
 		)
 	)
+	(label "IA18"
+		(at 207.01 41.91 180)
+		(effects
+			(font
+				(size 1.27 1.27)
+			)
+			(justify right bottom)
+		)
+	)
 	(label "P.D0"
 		(at 67.31 24.13 0)
@@
 		)
 	)
+	(label "IA17"
+		(at 207.01 39.37 180)
+		(effects
+			(font
+				(size 1.27 1.27)
+			)
+			(justify right bottom)
+		)
+	)
 	(label "PROT4"
 		(at 256.54 152.4 180)
 		(effects
 			(font
+				(size 1.27 1.27)
+			)
+			(justify right bottom)
+		)
+	)
+	(label "IA16"
+		(at 207.01 36.83 180)
+		(effects
+			(font
