File: schematics/kicad/sun2_mmu.kicad_sch (KiCad schematic)
At the start: 24 parts, among them U300 LS2518, U301 LS2518, U302 74F257, U303 2168, U304 2168, U305 2168, U306 2168, U307 2168, U308 2168, U309 2168, U310 2168, U313 74F08, U314 2949, U315 74F151, U316 P16R4, U317 2949, U318 2949, U319 2949, U320 2949, U321 74LS138, U322 74LS138, U323 74LS138, U324 74LS138

Commit message: Start global connections, error fixes
Connections:
- no-connect marks 8 -> 13
