File: schematics/kicad/sun2_periph.kicad_sch (KiCad schematic)
At the start: 29 parts, among them U203 74F74, U600 80287, U602 P16R4, U604 AM9513, U605 Z8530, U606 26LS32, U607 26LS32, U608 74LS04, U609 26LS29, U610 74LS04, U611 26LS29, U612 ICL7660, U613 74LS05, U614 ICL7660, U615 26LS32

Commit message: Finish connectors
Changed lines of the file:
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@@
-		)
-	)
-	(label "VEEB"
-		(at 200.66 151.13 0)
-		(effects
-			(font
-				(size 1.27 1.27)
-			)
-			(justify left bottom)
 		)
 	)
@@
 	(label "P.D1"
 		(at 102.87 29.21 0)
-		(effects
-			(font
-				(size 1.27 1.27)
-			)
-			(justify left bottom)
-		)
-	)
-	(label "VEEA"
-		(at 125.73 184.15 0)
 		(effects
 			(font
@@
 		)
 	)
+	(hierarchical_label "VEEB"
+		(shape output)
+		(at 198.12 151.13 0)
+		(effects
+			(font
+				(size 1.27 1.27)
+			)
+			(justify left)
+		)
+	)
 	(hierarchical_label "RTSA_"
 		(shape output)
@@
 		)
 	)
+	(hierarchical_label "VEEA"
+		(shape output)
+		(at 123.19 184.15 0)
+		(effects
+			(font
+				(size 1.27 1.27)
+			)
+			(justify left)
+		)
+	)

Commit message: Finish passives
Parts:
- removed unit 7 of U608
- removed unit 7 of U610
- removed unit 7 of U613
