File: schematics/kicad/sun2_periph.kicad_sch (KiCad schematic)
At the start: 29 parts, among them U203 74F74, U600 80287, U602 P16R4, U604 AM9513, U605 Z8530, U606 26LS32, U607 26LS32, U608 74LS04, U609 26LS29, U610 74LS04, U611 26LS29, U612 ICL7660, U613 74LS05, U614 ICL7660, U615 26LS32

Commit message: Start global connections, error fixes
Changed lines of the file:
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@@
 	(wire
 		(pts
+			(xy 135.89 99.06) (xy 135.89 101.6)
+		)
+		(stroke
+			(width 0)
+			(type default)
+		)
+	)
+	(wire
+		(pts
 			(xy 120.65 156.21) (xy 125.73 156.21)
 		)
@@
 		)
 	)
-	(label "IOACK"
-		(at 57.15 146.05 0)
-		(effects
-			(font
-				(size 1.27 1.27)
-			)
-			(justify left bottom)
-		)
-	)
 	(label "GND"
 		(at 39.37 71.12 180)
@@
 		)
 	)
-	(hierarchical_label "FPPERR\\"
-		(shape output)
-		(at 58.42 53.34 0)
+	(global_label "C.S7"
+		(shape input)
+		(at 41.91 158.75 180)
+		(fields_autoplaced yes)
 		(effects
 			(font
 				(size 1.27 1.27)
 			)
-			(justify left)
+			(justify right)
+		)
+		(property "Intersheetrefs" "${INTERSHEET_REFS}"
+			(at 34.631 158.75 0)
+			(effects
+				(font
+					(size 1.27 1.27)
+				)
+				(justify right)
+				(hide yes)
+			)
 		)
 	)
-	(hierarchical_label "VEEB"
-		(shape output)
-		(at 198.12 151.13 0)
+	(global_label "P.A[1..23]"
+		(shape input)
+		(at 165.1 58.42 180)
+		(fields_autoplaced yes)
 		(effects
 			(font
 				(size 1.27 1.27)
 			)
-			(justify left)
+			(justify right)
+		)
+		(property "Intersheetrefs" "${INTERSHEET_REFS}"
+			(at 152.6199 58.42 0)
+			(effects
+				(font
+					(size 1.27 1.27)
+				)
+				(justify right)
+				(hide yes)
+			)
 		)
 	)
-	(hierarchical_label "RTSA_"
-		(shape output)
-		(at 140.97 156.21 0)
+	(global_label "C(100.0-50)"
+		(shape input)
+		(at 40.64 172.72 180)
+		(fields_autoplaced yes)
 		(effects
 			(font
 				(size 1.27 1.27)
 			)
-			(justify left)
+			(justify right)
+		)
+		(property "Intersheetrefs" "${INTERSHEET_REFS}"
+			(at 25.2572 172.72 0)
+			(effects
+				(font
+					(size 1.27 1.27)
+				)
+				(justify right)
+				(hide yes)
+			)
 		)
 	)
-	(hierarchical_label "C(50.0-25)"
+	(global_label "C(50.0-25)"
 		(shape input)
 		(at 39.37 68.58 180)
+		(fields_autoplaced yes)
 		(effects
 			(font
@@
 			(justify right)
 		)
+		(property "Intersheetrefs" "${INTERSHEET_REFS}"
+			(at 25.1967 68.58 0)
+			(effects
+				(font
+					(size 1.27 1.27)
+				)
+				(justify right)
+				(hide yes)
+			)
+		)
 	)
-	(hierarchical_label "P.A[1..23]"
+	(global_label "C(100.0-50)"
 		(shape input)
-		(at 165.1 58.42 180)
+		(at 58.42 57.15 0)
+		(fields_autoplaced yes)
+		(effects
+			(font
+				(size 1.27 1.27)
+			)
+			(justify left)
+		)
+		(property "Intersheetrefs" "${INTERSHEET_REFS}"
+			(at 73.8028 57.15 0)
+			(effects
+				(font
+					(size 1.27 1.27)
+				)
+				(justify left)
+				(hide yes)
+			)
+		)
+	)
+	(global_label "P.D[0..15]"
+		(shape input)
+		(at 25.4 22.86 180)
+		(fields_autoplaced yes)
 		(effects
 			(font
@@
 			(justify right)
 		)
+		(property "Intersheetrefs" "${INTERSHEET_REFS}"
+			(at 12.7385 22.86 0)
+			(effects
+				(font
+					(size 1.27 1.27)
+				)
+				(justify right)
+				(hide yes)
+			)
+		)
 	)
-	(hierarchical_label "INT.SCC\\"
+	(global_label "P.FC2"
 		(shape input)
-		(at 177.8 71.12 180)
+		(at 111.76 106.68 180)
+		(fields_autoplaced yes)
 		(effects
 			(font
@@
 			(justify right)
 		)
+		(property "Intersheetrefs" "${INTERSHEET_REFS}"
+			(at 103.3319 106.68 0)
+			(effects
+				(font
+					(size 1.27 1.27)
+				)
+				(justify right)
+				(hide yes)
+			)
+		)
 	)
-	(hierarchical_label "DAB_"
+	(global_label "IOACK"
 		(shape output)
-		(at 215.9 107.95 0)
+		(at 57.15 146.05 0)
+		(fields_autoplaced yes)
 		(effects
 			(font
@@
 			(justify left)
 		)
+		(property "Intersheetrefs" "${INTERSHEET_REFS}"
+			(at 65.6991 146.05 0)
+			(effects
+				(font
+					(size 1.27 1.27)
+				)
+				(justify left)
+				(hide yes)
+			)
+		)
 	)
-	(hierarchical_label "DAA_"
+	(hierarchical_label "FPPERR\\"
 		(shape output)
-		(at 140.97 140.97 0)
+		(at 58.42 53.34 0)
 		(effects
 			(font
@@
 		)
 	)
-	(hierarchical_label "P.FC2"
+	(hierarchical_label "VEEB"
+		(shape output)
+		(at 198.12 151.13 0)
+		(effects
+			(font
+				(size 1.27 1.27)
+			)
+			(justify left)
+		)
+	)
+	(hierarchical_label "RTSA_"
+		(shape output)
+		(at 140.97 156.21 0)
+		(effects
+			(font
+				(size 1.27 1.27)
+			)
+			(justify left)
+		)
+	)
+	(hierarchical_label "INT.SCC\\"
 		(shape input)
-		(at 111.76 106.68 180)
+		(at 177.8 71.12 180)
 		(effects
 			(font
@@
 		)
 	)
+	(hierarchical_label "DAB_"
+		(shape output)
+		(at 215.9 107.95 0)
+		(effects
+			(font
+				(size 1.27 1.27)
+			)
+			(justify left)
+		)
+	)
+	(hierarchical_label "DAA_"
+		(shape output)
+		(at 140.97 140.97 0)
+		(effects
+			(font
+				(size 1.27 1.27)
+			)
+			(justify left)
+		)
+	)
 	(hierarchical_label "DCDA_"
 		(shape input)
@@
 		)
 	)
-	(hierarchical_label "C(100.0-50)"
-		(shape input)
-		(at 58.42 57.15 0)
-		(effects
-			(font
-				(size 1.27 1.27)
-			)
-			(justify left)
-		)
-	)
 	(hierarchical_label "WR.DCP\\"
 		(shape input)
@@
 		)
 	)
-	(hierarchical_label "C(100.0-50)"
-		(shape input)
-		(at 40.64 172.72 180)
-		(effects
-			(font
-				(size 1.27 1.27)
-			)
-			(justify right)
-		)
-	)
 	(hierarchical_label "DTRB_"
 		(shape output)
@@
 		)
 	)
-	(hierarchical_label "C.S7"
-		(shape input)
-		(at 41.91 158.75 180)
-		(effects
-			(font
-				(size 1.27 1.27)
-			)
-			(justify right)
-		)
-	)
 	(hierarchical_label "TXDA_"
 		(shape output)
@@
 		)
 	)
-	(hierarchical_label "P.D[0..15]"
-		(shape bidirectional)
-		(at 25.4 22.86 180)
-		(effects
-			(font
-				(size 1.27 1.27)
-			)
-			(justify right)
-		)
-	)
 	(hierarchical_label "RD.FPP\\"
 		(shape input)
@@
 					(unit 1)
 				)
+			)
+		)
+	)
+	(symbol
+		(lib_id "power:VCC")
+		(at 135.89 99.06 0)
+		(unit 1)
+		(exclude_from_sim no)
+		(in_bom yes)
+		(on_board yes)
+		(dnp no)
+		(fields_autoplaced yes)
+		(property "Reference" "#PWR036"
+			(at 135.89 102.87 0)
+			(effects
+				(font
+					(size 1.27 1.27)
+				)
+				(hide yes)
+			)
+		)
+		(property "Value" "VCC"
+			(at 135.89 93.98 0)
+			(effects
+				(font
+					(size 1.27 1.27)
+				)
+			)
+		)
+		(property "Footprint" ""
+			(at 135.89 99.06 0)
+			(effects
+				(font
+					(size 1.27 1.27)
+				)
+				(hide yes)
+			)
+		)
+		(property "Datasheet" ""
+			(at 135.89 99.06 0)
+			(effects
+				(font
+					(size 1.27 1.27)
+				)
+				(hide yes)
+			)
+		)
+		(property "Description" "Power symbol creates a global label with name \"VCC\""
+			(at 135.89 99.06 0)
+			(effects
+				(font
+					(size 1.27 1.27)
+				)
+				(hide yes)
+			)
+		)
+		(pin "1"
+		)
+		(instances
+			(project ""
+				(path "/67ee2072-0b57-4a50-8537-b17b5f651e89/8caf264c-65dd-4650-9fe1-d43351ee9f9b"
+					(reference "#PWR036")
+					(unit 1)
+				)
