File: schematics/kicad/sun2_rasterop_parity_p2.kicad_sch (KiCad schematic)
At the start: 18 parts, among them U101 74F32, U102 74F00, U109 74F08, U313 74F08, U422 74LS08, U500 74ALS244, U501 74ALS244, U502 74ALS244, U504 74ALS244, U505 74ALS244, U506 74ALS244, U507 74ALS244, U509 82S62, U510 82S62, U514 74F244, U515 74F244, U516 74F244, U517 74F244

Commit message: Rasterop, parity, P2 work
Parts:
- added U503: 74F32, Package_DIP:DIP-14_W7.62mm, symbol sun2:74F32
- added U508: 74F02, Package_DIP:DIP-14_W7.62mm, symbol sun2:74F02
- added U512: 74F74, Package_DIP:DIP-14_W7.62mm, symbol sun2:74F74
- added U513: 74F00, Package_DIP:DIP-14_W7.62mm, symbol sun2:74F00
- added U613: 74LS05, Package_DIP:DIP-14_W7.62mm, symbol 74xx:74LS05
Connections:
- net at U500.1 (OEa): now also U500.19 (OEb)
- net EN.PARERR: now reaches U422.10
- net at U422.8: now also U512.1 (~{R}), U512.13 (~{R})
- net at U422.9: now also U513.3
- net at U504.1 (OEa): now also U505.1 (OEa), U506.1 (OEa), U507.1 (OEa)
- net at U504.19 (OEb): now also U505.19 (OEb), U506.19 (OEb), U507.19 (OEb)
- net RD.RAM\: now reaches U109.12
- net RD.RAM\: now also U508.2, U508.5, U512.11 (C), U512.3 (C)
- net RD.ROP\: now reaches U109.13
- net at U509.5 (P9): now also U508.1
- net EN.PARGEN\: now reaches U509.8 (INH)
- net EN.PARGEN\: now also U510.8 (INH), U613.12
- net at U509.9 (EV): now also U503.12, U512.2 (D)
- net at U501.1 (OEa): now also U501.19 (OEb)
- net at U502.1 (OEa): now also U502.19 (OEb)
- net at U510.5 (P9): now also U508.4
- net at U510.9 (EV): now also U503.13, U512.12 (D)
- net R\/W: now reaches U102.1
- net DIS.D\: now reaches U102.2
- new net BERR: U513.1
- new net DS\: U513.2
- new net EN.PARGEN: U613.13
- new net P2.DOL: U508.3
- new net P2.DOU: U508.6
- new net PARERR: U503.11
- new net PARERRL\: U512.4 (~{S}), U512.6 (~{Q})
- new net PARERRU\: U512.10 (~{S}), U512.8 (~{Q})
Other:
- moved on the sheet: U101C, U422C, U500, U501, U502, U504, U505, U506, U507

Commit message: Completed Rasterop, parity, P2
Parts:
- added S500: 1KOhm, Resistor_THT:R_Array_SIP10, symbol Device:R_Network09_US
- added U206: 74F74, Package_DIP:DIP-14_W7.62mm, symbol sun2:74F74
- added U511: 16160 Rasterop, Package_DIP:DIP-28_W15.24mm, symbol sun2:16160
- added U518: 74S288, Package_DIP:DIP-16_W7.62mm, symbol sun2:74S288
- added U519: 74F374, Package_DIP:DIP-20_W7.62mm, symbol sun2:74F374
- added U520: 74LS20, Package_DIP:DIP-12_W7.62mm, symbol 74xx:74LS20
- added U610: 74LS04, Package_DIP:DIP-14_W7.62mm, symbol sun2:74LS04
Connections:
- net D0: now also U504.12 (O3a), U504.6 (I2a), U511.6 (D0)
- net D1: now also U504.16 (O1a), U504.2 (I0a), U511.7 (D1)
- net D10: now also U506.11 (I0b), U506.7 (O1b), U511.17 (D10)
- net D11: now also U506.15 (I2b), U506.3 (O3b), U511.18 (D11)
- net D12: now also U507.15 (I2b), U507.3 (O3b), U511.19 (D12)
- net D13: now also U507.11 (I0b), U507.7 (O1b), U511.20 (D13)
- net D14: now also U507.12 (O3a), U507.6 (I2a), U511.21 (D14)
- net D15: now also U507.16 (O1a), U507.2 (I0a), U511.22 (D15)
- net D2: now also U504.11 (I0b), U504.7 (O1b), U511.8 (D2)
- net D3: now also U504.15 (I2b), U504.3 (O3b), U511.9 (D3)
- net D4: now also U505.15 (I2b), U505.3 (O3b), U511.10 (D4)
- net D5: now also U505.11 (I0b), U505.7 (O1b), U511.11 (D5)
- net D6: now also U505.12 (O3a), U505.6 (I2a), U511.12 (D6)
- net D7: now also U505.16 (O1a), U505.2 (I0a), U206.12 (D), U511.13 (D7)
- net D8: now also U506.12 (O3a), U506.6 (I2a), U511.15 (D8)
- net D9: now also U506.16 (O1a), U506.2 (I0a), U511.16 (D9)
- net DIS.D\: now also S500.3 (R2), U519.19 (Q8)
- net GND: now also U500.10 (GND), U501.10 (GND), U502.1 (OEa), U502.10 (GND), U502.19 (OEb), U504.10 (GND), U505.10 (GND), U506.10 (GND), U507.10 (GND), U511.14 (GND), U511.5 (CS), U518.15 (S0), U518.8 (GND), U519.10 (GND)
- net RD.RAM\: now also U313.5
- net RD.ROP\: now also U511.27 (RD)
- net R\/W: now also U513.5, U520.13
- net VCC: now also U500.20 (VCC), U501.20 (VCC), U502.20 (VCC), U504.20 (VCC), U505.20 (VCC), U506.20 (VCC), U507.20 (VCC), S500.1 (common), U206.10 (~{S}), U511.28 (VCC), U518.16 (VCC), U519.20 (VCC)
- net C.S3: now reaches U500.1 (OEa), U500.19 (OEb)
- net P.A3: now reaches U500.11 (I0b)
- net P.A3: now also U511.3 (A2), U520.4
- net P2.A7: now reaches U500.12 (O3a)
- net P2.A7: now also U501.12 (O3a)
- net P.A6: now reaches U500.13 (I1b)
- net P2.A2: now reaches U500.14 (O2a)
- net P2.A2: now also U501.14 (O2a)
- net P.A4: now reaches U500.15 (I2b)
- net P.A4: now also U511.4 (A3), U520.5
- net P2.A8: now reaches U500.16 (O1a)
- net P2.A8: now also U501.16 (O1a)
- net P.A5: now reaches U500.17 (I3b)
- net P2.A1: now reaches U500.18 (O0a)
- net P2.A1: now also U501.18 (O0a)
- net P.A1: now reaches U500.2 (I0a)
- net P.A1: now also U511.1 (A0), U520.1
- net P2.A5: now reaches U500.3 (O3b)
- net P2.A5: now also U501.3 (O3b)
- net P.A8: now reaches U500.4 (I1a)
- net P2.A4: now reaches U500.5 (O2b)
- net P2.A4: now also U501.5 (O2b)
- net P.A2: now reaches U500.6 (I2a)
- net P.A2: now also U511.2 (A1), U520.2
- net P2.A6: now reaches U500.7 (O1b)
- net P2.A6: now also U501.7 (O1b)
- net P.A7: now reaches U500.8 (I3a)
- net P2.A3: now reaches U500.9 (O0b)
- net P2.A3: now also U501.9 (O0b)
- net P2.R/W\: now reaches U504.1 (OEa), U505.1 (OEa), U506.1 (OEa), U507.1 (OEa)
- net P2.R/W\: now also U513.6
- net P2.DO2: now reaches U504.13 (I1b)
- net P2.DI0: now reaches U504.14 (O2a)
- net P2.DO3: now reaches U504.17 (I3b)
- net P2.DI1: now reaches U504.18 (O0a)
- net at U504.19 (OEb), U505.19 (OEb), U506.19 (OEb)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: now also U313.6
- net P2.DO1: now reaches U504.4 (I1a)
- net P2.DI3: now reaches U504.5 (O2b)
- net P2.DO0: now reaches U504.8 (I3a)
- net P2.DI2: now reaches U504.9 (O0b)
- net P.AS\: now reaches U503.10
- net RAS\: now reaches U503.8
- net RAS\: now also U502.4 (I1a)
- net at U503.9: now also U513.8
- net P2.DO10: now reaches U506.13 (I1b)
- net P2.DI8: now reaches U506.14 (O2a)
- net P2.DO11: now reaches U506.17 (I3b)
- net P2.DI9: now reaches U506.18 (O0a)
- net P2.DO9: now reaches U506.4 (I1a)
- net P2.DI11: now reaches U506.5 (O2b)
- net P2.DO8: now reaches U506.8 (I3a)
- net P2.DI10: now reaches U506.9 (O0b)
- net P2.DO13: now reaches U507.13 (I1b)
- net P2.DI14: now reaches U507.14 (O2a)
- net P2.DO12: now reaches U507.17 (I3b)
- net P2.DI15: now reaches U507.18 (O0a)
- net P2.DO15: now reaches U507.4 (I1a)
- net P2.DI12: now reaches U507.5 (O2b)
- net P2.DO14: now reaches U507.8 (I3a)
- net P2.DI13: now reaches U507.9 (O0b)
- net at U513.11: now also U513.10, U513.9
- net C.S7: now reaches U513.12
- net SYSB: now reaches U513.13
- net C.S3\: now reaches U501.1 (OEa), U501.19 (OEb)
- net MA11: now reaches U501.11 (I0b)
- net MA14: now reaches U501.13 (I1b)
- net MA12: now reaches U501.15 (I2b)
- net MA13: now reaches U501.17 (I3b)
- net MA17: now reaches U501.2 (I0a)
- net MA16: now reaches U501.4 (I1a)
- net P.A10: now reaches U501.6 (I2a)
- net MA15: now reaches U501.8 (I3a)
- net MA19: now reaches U502.11 (I0b)
- net P2.CAS\: now reaches U502.12 (O3a)
- net MA22: now reaches U502.13 (I1b)
- net P2.A18: now reaches U502.14 (O2a)
- net MA20: now reaches U502.15 (I2b)
- net P2.RAS\: now reaches U502.16 (O1a)
- net MA21: now reaches U502.17 (I3b)
- net P2.A9: now reaches U502.18 (O0a)
- net P.A9: now reaches U502.2 (I0a)
- net P2.A21: now reaches U502.3 (O3b)
- net P2.A20: now reaches U502.5 (O2b)
- net MA18: now reaches U502.6 (I2a)
- net P2.A22: now reaches U502.7 (O1b)
- net C.S4\: now reaches U502.8 (I3a)
- net P2.A19: now reaches U502.9 (O0b)
- net LD.DST\: now reaches U513.4
- net LD.DST\: now also U313.4, S500.7 (R6), U511.25 (DST), U519.15 (Q6)
- net P2.DO5: now reaches U505.13 (I1b)
- net P2.DI6: now reaches U505.14 (O2a)
- net P2.DO4: now reaches U505.17 (I3b)
- net P2.DI7: now reaches U505.18 (O0a)
- net P2.DO7: now reaches U505.4 (I1a)
- net P2.DI4: now reaches U505.5 (O2b)
- net P2.DO6: now reaches U505.8 (I3a)
- net P2.DI5: now reaches U505.9 (O0b)
- net at U101.10: now also U520.6
- net at U101.8: now also U206.11 (C)
- net WR.ROP\: now reaches U101.9
- net WR.ROP\: now also U511.26 (WR)
- net P.UDS\: now reaches U503.4
- net WR.M\: now reaches U503.5
- net WR.M\: now also U503.2, S500.8 (R7), U518.13 (A3), U519.9 (Q4)
- net P2.WEU\: now reaches U503.6
- net P.LDS\: now reaches U503.1
- net P2.WEL\: now reaches U503.3
- new net: U518.5 (Q4), U519.13 (D5)
- new net: U518.6 (Q5), U519.14 (D6)
- new net: U518.7 (Q6), U519.17 (D7)
- new net: U518.9 (Q7), U519.18 (D8)
- new net: U518.1 (Q0), U519.3 (D1)
- new net: U518.2 (Q1), U519.4 (D2)
- new net: U518.3 (Q2), U519.7 (D3)
- new net: U518.4 (Q3), U519.8 (D4)
- new net C(100.50-0): U519.11 (CLK)
- new net DIS\: U520.9
- new net LD.SRC\: S500.9 (R8), U511.24 (SRC), U519.12 (Q5)
- new net OE.ROP\: S500.5 (R4), U511.23 (OE), U519.16 (Q7)
- new net P.FC2: U610.11
- new net P.FC2\: U520.10, U610.10
- new net P.RESET\: U206.13 (~{R})
- new net P2.WAIT\: S500.10 (R9)
- new net ROP: U206.9 (Q), U520.12
- new net ROPCYC\: U518.14 (A4), U520.8
- new net ROPST0: S500.2 (R1), U518.10 (A0), U519.2 (Q1)
- new net ROPST1: S500.4 (R3), U518.11 (A1), U519.5 (Q2)
- new net ROPST2: S500.6 (R5), U518.12 (A2), U519.6 (Q3)
- new net WR.RAM\: U519.1 (OE)
Other:
- moved on the sheet: U101C, U313B, U422C, U500, U501, U502, U503A, U503B, U503C, U503D, U504, U505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

Commit message: Serials
Other:
- note added: "P2 BUS INTERFACE"
- note added: "PARITY LOGIC"
- note added: "RASTEROP PROCESSOR"
Changed lines of the file:
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@@
 	(generator_version "9.0")
 	(paper "USLetter")
+	(text "P2 BUS INTERFACE"
+		(exclude_from_sim no)
+		(at 231.14 14.986 0)
+		(effects
+			(font
+				(size 1.27 1.27)
+				(thickness 0.254)
+				(bold yes)
+			)
+		)
+	)
+	(text "RASTEROP PROCESSOR"
+		(exclude_from_sim no)
+		(at 57.912 14.986 0)
+		(effects
+			(font
+				(size 1.27 1.27)
+				(thickness 0.254)
+				(bold yes)
+			)
+		)
+	)
+	(text "PARITY LOGIC"
+		(exclude_from_sim no)
+		(at 151.638 15.24 0)
+		(effects
+			(font
+				(size 1.27 1.27)
+				(thickness 0.254)
+				(bold yes)
+			)
+		)
+	)
 	(junction
 		(at 45.72 96.52)
