File: schematics/kicad/sun2_rasterop_parity_p2.kicad_sch (KiCad schematic)
At the start: 30 parts, among them U101 74F32, U102 74F00, U109 74F08, U206 74F74, U313 74F08, U422 74LS08, U500 74ALS244, U501 74ALS244, U502 74ALS244, U503 74F32, U504 74ALS244, U505 74ALS244, U506 74ALS244, U507 74ALS244, U508 74F02, U509 82S62, U510 82S62, U511 16160 Rasterop, U512 74F74, U513 74F00, U514 74F244, U515 74F244, U516 74F244, U517 74F244, U518 74S288, U519 74F374, U520 74LS20, U610 74LS04, U613 74LS05

Commit message: P1 and P2 connectors
Connections:
- net P2.DIL: now reaches U509.6 (OD)
- net P2.DIU: now reaches U510.6 (OD)
Changed lines of the file:
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@@
+		)
+	)
+	(hierarchical_label "P2.DIU"
+		(shape output)
+		(at 142.24 82.55 0)
+		(effects
+			(font
+				(size 1.27 1.27)
+			)
+			(justify left)
 		)
 	)
@@
 		)
 	)
+	(hierarchical_label "P2.DIL"
+		(shape output)
+		(at 142.24 40.64 0)
+		(effects
+			(font
+				(size 1.27 1.27)
+			)
+			(justify left)
+		)
+	)

Commit message: Finish passives
Parts:
- removed unit 5 of U503
- removed unit 5 of U508
- removed unit 3 of U512
- removed unit 5 of U513
- removed unit 3 of U520
Connections:
- no-connect marks 0 -> 6
Other:
- moved on the sheet: U508C, U508D
