File: schematics/kicad/sun2_rasterop_parity_p2.kicad_sch (KiCad schematic)
At the start: 30 parts, among them U101 74F32, U102 74F00, U109 74F08, U206 74F74, U313 74F08, U422 74LS08, U500 74ALS244, U501 74ALS244, U502 74ALS244, U503 74F32, U504 74ALS244, U505 74ALS244, U506 74ALS244, U507 74ALS244, U508 74F02, U509 82S62, U510 82S62, U511 16160 Rasterop, U512 74F74, U513 74F00, U514 74F244, U515 74F244, U516 74F244, U517 74F244, U518 74S288, U519 74F374, U520 74LS20, U610 74LS04, U613 74LS05

Commit message: Start global connections, error fixes
Connections:
- net C.S3\ is gone; now on net C.S3: U501.1 (OEa), U501.19 (OEb)
- no-connect marks 6 -> 7
