File: schematics/kicad/sun2.kicad_sch (KiCad schematic)
At the start: 0 parts

Commit message: Start global connections, error fixes
Other:
- sheet ADDRS_BUFFERS ports: added AEN\, BEN\, CE.BYTE\, CE.WORD\, IORC\, IOWC\, LDS, MRDC\, MWTC\, P.LDS\, P1.A\[0..19], P1.BCLK\, P1.BHEN\, P1.BPRN\, P1.BPRO\, P1.BREQ\, P1.BUSY\, P1.CBRQ\, P1.CCLK\, P1.D\[0..15], P1.INIT\, P1.IORC\, P1.IOWC\, P1.MRDC\, P1.MWTC\, P1.XACK\, P1TOP\, Q.AS\, RREQ\, SYSB, UDS, XACK\, XEN\; removed none
- sheet CLOCK_DVMA ports: added AEN\, AS, BEN\, CE.BYTE\, CE.WORD\, DIS\, EN.DVMA, EN.S4, INIT\, IORC\, MRDC\, P.AS\, P.BACK\, P.BG\, P.BR\, P.HALT\, P.LDS\, P.R/W\, P.UDS\, P1.A\[0..19], P1.BHEN\, P1.MRDC\, P1.MRWC\, P1.MWTC\, P1.XACK\, P1TOP\, PARERR, POR\, PROTERR\, Q.AS\, REN\, SACK\, SAS\, SYSB, TIMEOUT\, VALID, XBERR\, XEN\, XHALT\, XREQ\; removed none
- sheet CONNECTORS ports: added CTSA_, CTSB_, DAA_, DAB_, DBA_, DBB_, DCDA_, DCDB_, DDA_, DDB_, DSRA_, DSRB_, DTRA_, DTRB_, INT1\, INT2\, INT3\, INT4\, INT5\, INT6\, INT7\, P.HALT\, P.RESET\, P1.A\[0..19], P1.BCLK\, P1.BHEN\, P1.BPRN\, P1.BPRO\, P1.BREQ\, P1.BUSY\, P1.CBRQ\, P1.CCLK\, P1.D\[0..15], P1.INIT\, P1.IORC\, P1.IOWC\, P1.MRDC\, P1.MWTC\, P1.XACK\, P2.CAS\, P2.DIL, P2.DIU, P2.DI[0..15], P2.DOL, P2.DOU, P2.DO[0..15], P2.RAS\, P2.R/W\, P2.WAIT\, P2.WEL\, P2.WEU\, POR\, RD.PORT\, REN\, RTSA_, RTSB_, RXDA_, RXDB_, TXDA_, TXDB_, VEEA, VEEB, WR.DIAG\, {P2.A[1..9] P2.A[18..22]}; removed none
- sheet CPU ports: added AS, BERR, DS\, EN.INT, EN.INT1, EN.INT2, EN.INT3, EN.PARGEN\, EN.S4, ERR, ERR\, FPPERR\, INIT\, INT.SCC\, INT1\, INT2\, INT3\, INT4\, INT5\, INT6\, INT7\, LDS, OE.ROP\, P.AS\, P.BACK\, P.BG\, P.BR\, P.HALT\, P.LDS\, P.RESET\, P.R/W\, P.UDS\, P.VPA\, P1.INIT\, P2.WAIT\, PARERRL\, PARERRU\, POR\, PROTERR\, Q.AS\, RESET, ROPCYC\, TIMEOUT\, UDS, XACK, XACK\, XBERR\, XHALT\; removed none
- sheet MMU ports: added BOOTEN\, DIS\, DS\, ERR\, LDS, P.AS\, P.BACK\, P.INTA\, P.R/W\, P.SPROG\, RD.ENABLE\, RD.ERROR\, RD.IDPROM\, UDS, VALID, WR.DIAG\, WR.ENABLE\; removed none
- sheet PERIPHERALS ports: added CTSA_, CTSB_, DAA_, DAB_, DBA_, DBB_, DCDA_, DCDB_, DDA_, DDB_, DSRA_, DSRB_, DTRA_, DTRB_, FPPERR\, INT.SCC\, INT5\, INT7\, RD.DCP\, RD.FPP\, RD.SCC\, RD.TIMER\, RESET, RTSA_, RTSB_, RXDA_, RXDB_, TXDA_, TXDB_, VEEA, VEEB, WD.SCC\, WR.DCP\, WR.FPP\, WR.TIMER\; removed none
- sheet PROM_RTC_REGS ports: added AEN\, BERR, BOOTEN\, DS\, EN.DVMA, EN.INT, EN.INT1, EN.INT2, EN.INT3, EN.PARERR, EN.PARGEN, ERR, INIT\, IORC\, IOWC\, MRDC\, MWTC\, P.INTA\, P.SPROG\, P.VPA\, PARERRL\, PARERRU\, POR\, PROTERR\, RD.DCP\, RD.ENABLE\, RD.ERROR\, RD.FPP\, RD.IDPROM\, RD.IO\, RD.PORT\, RD.RAM\, RD.ROP\, RD.SCC\, RD.TIMER\, TIMEOUT\, WR.DCP\, WR.ENABLE\, WR.FPP\, WR.IO\, WR.RAM\, WR.ROP\, WR.SCC\, WR.TIMER\; removed none
- sheet RASTEROP_PARITY_P2 ports: added BERR, DIS\, DS\, EN.PARERR, EN.PARGEN, EN.PARGEN\, P.AS\, P.LDS\, P.RESET\, P.UDS\, P2.CAS\, P2.DIL, P2.DIU, P2.DI[0..15], P2.DOL, P2.DOU, P2.DO[0..15], P2.RAS\, P2.R/W\, P2.WAIT\, P2.WEL\, P2.WEU\, PARERR, PARERRL\, PARERRU\, RD.RAM\, RD.ROP\, ROPCYC\, SYSB, WR.RAM\, WR.ROP\, {P2.A[1..9] P2.A[18..22]}; removed none
