File: schematics/kicad/sun2_clock.kicad_sch (KiCad schematic)
At the start: 14 parts, among them U102 74F00, U200 20Mhz, U201 74F74, U203 74F74, U204 74F74, U205 74F74, U207 74F74, U209 74LS393, U210 74LS491, U211 P20X10, U212 P20L10, U213 P16R4, U313 74F08, U703 74F08

Commit message: Finish passives
Parts:
- removed unit 3 of U201
- removed unit 3 of U203
- removed unit 3 of U204
- removed unit 3 of U205
- removed unit 3 of U207
- removed unit 2 of U209
- removed unit 2 of U211
- removed unit 5 of U313
- removed unit 5 of U703
Connections:
- no-connect marks 9 -> 12
Other:
- moved on the sheet: U313C

Commit message: Start global connections, error fixes
Connections:
- no-connect marks 12 -> 13
