File: schematics/kicad/sun2_connectors.kicad_sch (KiCad schematic)
At the start: 4 parts, among them J1 Conn_02x25_Odd_Even, J2 Conn_02x25_Odd_Even, P1 2x43 connector, P2 Connector 2x30

Commit message: P1 and P2 connectors
Connections:
- net P2.A18: now also P2.2
- net P2.A2: now also P2.19
- net P2.A20: now also P2.4
- net P2.A21: now also P2.14
- net P2.A22: now also P2.20
- net P2.A3: now also P2.25
- net P2.A4: now also P2.31
- net P2.A5: now also P2.37
- net P2.A6: now also P2.43
- net P2.A7: now also P2.49
- net P2.A8: now also P2.55
- net P2.DI10: now also P2.45
- net P2.DI11: now also P2.47
- net P2.DI12: now also P2.51
- net P2.DI13: now also P2.53
- net P2.DI14: now also P2.57
- net P2.DI15: now also P2.59
- net P2.DI3: now also P2.17
- net P2.DI4: now also P2.21
- net P2.DI5: now also P2.23
- net P2.DI6: now also P2.27
- net P2.DI7: now also P2.29
- net P2.DI8: now also P2.39
- net P2.DI9: now also P2.41
- net P2.DO0: now also P2.10
- net P2.DO1: now also P2.12
- net P2.DO10: now also P2.46
- net P2.DO11: now also P2.48
- net P2.DO12: now also P2.52
- net P2.DO13: now also P2.54
- net P2.DO14: now also P2.58
- net P2.DO15: now also P2.60
- net P2.DO2: now also P2.16
- net P2.DO3: now also P2.18
- net P2.DO4: now also P2.22
- net P2.DO5: now also P2.24
- net P2.DO6: now also P2.28
- net P2.DO7: now also P2.30
- net P2.DO8: now also P2.40
- net P2.DO9: now also P2.42
- net P2.RAS\: now also P2.6
- net GND: now reaches P1.1
- net GND: now also P1.11, P1.12, P1.2, P1.75, P1.76, P1.85, P1.86, P2.32, P2.38, P2.44
- net P1.BCLK\: now reaches P1.13
- net P1.INIT\: now reaches P1.14
- net P1.BPRN\: now reaches P1.15
- net P1.BPRO\: now reaches P1.16
- net P1.BUSY\: now reaches P1.17
- net P1.BREQ\: now reaches P1.18
- net P1.MRDC\: now reaches P1.19
- net P1.MWTC\: now reaches P1.20
- net P1.IORC\: now reaches P1.21
- net P1.IOWC\: now reaches P1.22
- net P1.XACK\: now reaches P1.23
- net P1.INH1\: now reaches P1.24
- net P1.AACK\: now reaches P1.25
- net P1.INH2\: now reaches P1.26
- net P1.BHEN\: now reaches P1.27
- net P1.A\16: now reaches P1.28
- net P1.CBRQ\: now reaches P1.29
- net VCC: now reaches P1.3
- net VCC: now also P1.4, P1.5, P1.6, P1.81, P1.82, P1.83, P1.84
- net P1.A\17: now reaches P1.30
- net P1.CCLK\: now reaches P1.31
- net P1.A\18: now reaches P1.32
- net P1.INTA\: now reaches P1.33
- net P1.A\19: now reaches P1.34
- net INT6\: now reaches P1.35
- net INT7\: now reaches P1.36
- net INT4\: now reaches P1.37
- net INT5\: now reaches P1.38
- net INT2\: now reaches P1.39
- net INT3\: now reaches P1.40
- net P1.INT0\: now reaches P1.41
- net INT1\: now reaches P1.42
- net P1.A\14: now reaches P1.43
- net P1.A\15: now reaches P1.44
- net P1.A\12: now reaches P1.45
- net P1.A\13: now reaches P1.46
- net P1.A\10: now reaches P1.47
- net P1.A\11: now reaches P1.48
- net P1.A\8: now reaches P1.49
- net P1.A\9: now reaches P1.50
- net P1.A\6: now reaches P1.51
- net P1.A\7: now reaches P1.52
- net P1.A\4: now reaches P1.53
- net P1.A\5: now reaches P1.54
- net P1.A\2: now reaches P1.55
- net P1.A\3: now reaches P1.56
- net P1.A\0: now reaches P1.57
- net P1.A\1: now reaches P1.58
- net P1.D\14: now reaches P1.59
- net P1.D\15: now reaches P1.60
- net P1.D\12: now reaches P1.61
- net P1.D\13: now reaches P1.62
- net P1.D\10: now reaches P1.63
- net P1.D\11: now reaches P1.64
- net P1.D\8: now reaches P1.65
- net P1.D\9: now reaches P1.66
- net P1.D\6: now reaches P1.67
- net P1.D\7: now reaches P1.68
- net P1.D\4: now reaches P1.69
- net P1.D\5: now reaches P1.70
- net P1.D\2: now reaches P1.71
- net P1.D\3: now reaches P1.72
- net P1.D\0: now reaches P1.73
- net P1.D\1: now reaches P1.74
- net REN\: now reaches P2.26
- net P2.DIL: now reaches P2.33
- net P2.DOL: now reaches P2.34
- net P2.DIU: now reaches P2.35
- net P2.DOU: now reaches P2.36
- net P2.R/W\: now reaches P2.50
- net P2.WEU\: now reaches P2.56
- net P2.WEL\: now reaches P2.8
- no-connect marks 0 -> 8

Commit message: Finish connectors
Parts:
- added J803, J804: LED_Block, Connector_PinHeader_1.00mm:PinHeader_2x04_P1.00mm_Vertical, symbol sun2:LED_Block
- added R800, R801: 1k, symbol Device:R_Small_US
- added S800, S801: 4.7KOhm, Resistor_THT:R_Array_SIP10, symbol Device:R_Network09_US
- added U1: 74LS273, symbol 74xx:74LS273
- added U800, U801: 74LS244, Package_DIP:DIP-20_W7.62mm, symbol sun2:74LS244
Connections:
- net GND: now also J1.13 (Pin_13), J1.38 (Pin_38), J2.10 (Pin_10), J2.12 (Pin_12), J2.14 (Pin_14), J2.16 (Pin_16), J2.18 (Pin_18), J2.2 (Pin_2), J2.20 (Pin_20), J2.22 (Pin_22), J2.24 (Pin_24), J2.26 (Pin_26), J2.28 (Pin_28), J2.30 (Pin_30), J2.32 (Pin_32), J2.34 (Pin_34), J2.36 (Pin_36), J2.38 (Pin_38), J2.4 (Pin_4), J2.40 (Pin_40), J2.42 (Pin_42), J2.44 (Pin_44), J2.46 (Pin_46), J2.48 (Pin_48), J2.50 (Pin_50), J2.6 (Pin_6), J2.8 (Pin_8), U1.10 (GND), U800.10 (GND), U801.10 (GND)
- net INT7\: now also J2.41 (Pin_41)
- net VCC: now also J2.37 (Pin_37), J2.39 (Pin_39), J2.49 (Pin_49), J803.1 (A), J803.3 (A), J803.5, J803.7, J804.1 (A), J804.3 (A), J804.5, J804.7, S800.1 (common), S801.1 (common), U1.20 (VCC), U800.20 (VCC), U801.20 (VCC)
- net DSRA_: now reaches J1.11 (Pin_11)
- net DTRA_: now reaches J1.14 (Pin_14)
- net DCDA_: now reaches J1.15 (Pin_15)
- net DAA_: now reaches J1.22 (Pin_22)
- net SPAREA_: now reaches J1.24 (Pin_24)
- net SPAREA_: now also R800.2
- net TXDB_: now reaches J1.28 (Pin_28)
- net DBB_: now reaches J1.29 (Pin_29)
- net TXDA_: now reaches J1.3 (Pin_3)
- net RXDB_: now reaches J1.30 (Pin_30)
- net RTSB_: now reaches J1.32 (Pin_32)
- net DDB_: now reaches J1.33 (Pin_33)
- net CTSB_: now reaches J1.34 (Pin_34)
- net DSRB_: now reaches J1.36 (Pin_36)
- net DTRB_: now reaches J1.39 (Pin_39)
- net DBA_: now reaches J1.4 (Pin_4)
- net DCDB_: now reaches J1.40 (Pin_40)
- net DAB_: now reaches J1.47 (Pin_47)
- net SPAREB_: now reaches J1.49 (Pin_49)
- net SPAREB_: now also R801.2
- net RXDA_: now reaches J1.5 (Pin_5)
- net RTSA_: now reaches J1.7 (Pin_7)
- net DDA_: now reaches J1.8 (Pin_8)
- net CTSA_: now reaches J1.9 (Pin_9)
- net IN0_: now reaches J2.1 (Pin_1)
- net IN0_: now also S800.4 (R3), U800.2 (I0a)
- net IN5_: now reaches J2.11 (Pin_11)
- net IN5_: now also S800.9 (R8), U800.13 (I1b)
- net IN6_: now reaches J2.13 (Pin_13)
- net IN6_: now also S800.10 (R9), U800.8 (I3a)
- net IN7_: now reaches J2.15 (Pin_15)
- net IN7_: now also S801.2 (R1), U800.11 (I0b)
- net IN8_: now reaches J2.17 (Pin_17)
- net IN8_: now also S801.3 (R2), U801.2 (I0a)
- net IN9_: now reaches J2.19 (Pin_19)
- net IN9_: now also S801.4 (R3), U801.17 (I3b)
- net IN10_: now reaches J2.21 (Pin_21)
- net IN10_: now also S801.5 (R4), U801.4 (I1a)
- net IN11_: now reaches J2.23 (Pin_23)
- net IN11_: now also S801.6 (R5), U801.15 (I2b)
- net IN12_: now reaches J2.25 (Pin_25)
- net IN12_: now also S801.7 (R6), U801.6 (I2a)
- net IN13_: now reaches J2.27 (Pin_27)
- net IN13_: now also S801.8 (R7), U801.13 (I1b)
- net IN14_: now reaches J2.29 (Pin_29)
- net IN14_: now also S801.9 (R8), U801.8 (I3a)
- net IN1_: now reaches J2.3 (Pin_3)
- net IN1_: now also S800.5 (R4), U800.17 (I3b)
- net IN15_: now reaches J2.31 (Pin_31)
- net IN15_: now also S801.10 (R9), U801.11 (I0b)
- net POR\: now reaches J2.43 (Pin_43)
- net P.RESET\: now reaches J2.45 (Pin_45)
- net P.RESET\: now also U1.1 (~{Mr})
- net P.HALT\: now reaches J2.47 (Pin_47)
- net IN2_: now reaches J2.5 (Pin_5)
- net IN2_: now also S800.6 (R5), U800.4 (I1a)
- net IN3_: now reaches J2.7 (Pin_7)
- net IN3_: now also S800.7 (R6), U800.15 (I2b)
- net IN4_: now reaches J2.9 (Pin_9)
- net IN4_: now also S800.8 (R7), U800.6 (I2a)
- new net LED0: J803.2 (K), U1.2 (Q0)
- new net LED1: J803.4, U1.19 (Q7)
- new net LED2: J803.6 (K), U1.5 (Q1)
- new net LED3: J803.8 (K), U1.16 (Q6)
- new net LED4: J804.2 (K), U1.6 (Q2)
- new net LED5: J804.4, U1.15 (Q5)
- new net LED6: J804.6 (K), U1.9 (Q3)
- new net LED7: J804.8 (K), U1.12 (Q4)
- new net P.D0: U1.3 (D0), U800.18 (O0a)
- new net P.D1: U1.18 (D7), U800.3 (O3b)
- new net P.D10: U801.16 (O1a)
- new net P.D11: U801.5 (O2b)
- new net P.D12: U801.14 (O2a)
- new net P.D13: U801.7 (O1b)
- new net P.D14: U801.12 (O3a)
- new net P.D15: U801.9 (O0b)
- new net P.D2: U1.4 (D1), U800.16 (O1a)
- new net P.D3: U1.17 (D6), U800.5 (O2b)
- new net P.D4: U1.7 (D2), U800.14 (O2a)
- new net P.D5: U1.14 (D5), U800.7 (O1b)
- new net P.D6: U1.8 (D3), U800.12 (O3a)
- new net P.D7: U1.13 (D4), U800.9 (O0b)
- new net P.D8: U801.18 (O0a)
- new net P.D9: U801.3 (O3b)
- new net RD.PORT\: U800.1 (OEa), U800.19 (OEb), U801.1 (OEa), U801.19 (OEb)
- new net VEEA: R800.1
- new net VEEB: R801.1
- new net WR.DIAG\: U1.11 (Cp)
- no-connect marks 8 -> 38
Other:
- moved on the sheet: J1, J2, P1, P2
