File: schematics/kicad/sun2_cpu.kicad_sch (KiCad schematic)
At the start: 22 parts, among them U100 MC68010, U102 74F00, U109 74F08, U110 7407, U111 74F251, U114 74LS20, U115 74F04, U119 74LS148, U120 8211, U122 7406, U206 74F74, U608 74LS04, U610 74LS04

Commit message: Completed Rasterop, parity, P2
Parts:
- removed unit 2 of U206
- U608, U610: footprint (none) -> Package_DIP:DIP-14_W7.62mm; Order Link (none) -> https://www.digikey.com/en/products/detail/texas-instrument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
Changed lines of the file:
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@@
 		)
 	)
-	(label "P.RESET\\"
-		(at 121.92 189.23 0)
-		(effects
-			(font
-				(size 1.27 1.27)
-			)
-			(justify left bottom)
-		)
-	)
 	(label "INT6\\"
 		(at 66.04 176.53 0)
@@
 		)
 	)
+	(hierarchical_label "P.RESET\\"
+		(shape output)
+		(at 129.54 189.23 180)
+		(effects
+			(font
+				(size 1.27 1.27)
+			)
+			(justify right)
+		)
+	)
 	(hierarchical_label "FPPERR\\"
 		(shape input)
@@
 			)
 		)
-		(property "Footprint" ""
+		(property "Footprint" "Package_DIP:DIP-14_W7.62mm"
 			(at 172.72 165.1 0)
 			(effects
@@
 			)
 		)
+		(property "Order Link" "https://www.digikey.com/en/products/detail/texas-instruments/SN74LS04N/277275"
+			(at 172.72 165.1 0)
+			(effects
+				(font
+					(size 1.27 1.27)
+				)
+				(hide yes)
+			)
+		)
 		(pin "1"
 		)
@@
 			)
 		)
-		(property "Footprint" ""
+		(property "Footprint" "Package_DIP:DIP-14_W7.62mm"
 			(at -29.21 132.08 0)
 			(effects
@@
 			)
 		)
+		(property "Order Link" "https://www.digikey.com/en/products/detail/texas-instruments/SN74LS04N/277275"
+			(at -29.21 132.08 0)
+			(effects
+				(font
+					(size 1.27 1.27)
+				)
+				(hide yes)
+			)
+		)
 		(pin "3"
 		)
@@
 			)
 		)
-		(property "Footprint" ""
+		(property "Footprint" "Package_DIP:DIP-14_W7.62mm"
 			(at -29.21 123.19 0)
 			(effects
@@
 			)
 		)
+		(property "Order Link" "https://www.digikey.com/en/products/detail/texas-instruments/SN74LS04N/277275"
+			(at -29.21 123.19 0)
+			(effects
+				(font
+					(size 1.27 1.27)
+				)
+				(hide yes)
+			)
+		)
 		(pin "3"
 		)
@@
 			)
 		)
-		(property "Footprint" ""
+		(property "Footprint" "Package_DIP:DIP-14_W7.62mm"
 			(at -29.21 113.03 0)
 			(effects
@@
 			)
 		)
+		(property "Order Link" "https://www.digikey.com/en/products/detail/texas-instruments/SN74LS04N/277275"
+			(at -29.21 113.03 0)
+			(effects
+				(font
+					(size 1.27 1.27)
+				)
+				(hide yes)
+			)
+		)
 		(pin "3"
 		)
@@
 			)
 		)
-		(property "Footprint" ""
+		(property "Footprint" "Package_DIP:DIP-14_W7.62mm"
 			(at 59.69 226.06 0)
 			(effects
@@
 			)
 		)
+		(property "Order Link" "https://www.digikey.com/en/products/detail/texas-instruments/SN74LS04N/277275"
+			(at 59.69 226.06 0)
+			(effects
+				(font
+					(size 1.27 1.27)
+				)
+				(hide yes)
+			)
+		)
 		(pin "1"
 		)
@@
 			)
 		)
-		(property "Footprint" ""
+		(property "Footprint" "Package_DIP:DIP-14_W7.62mm"
 			(at 186.69 233.68 0)
 			(effects
@@
 			)
 		)
+		(property "Order Link" "https://www.digikey.com/en/products/detail/texas-instruments/SN74LS04N/277275"
+			(at 186.69 233.68 0)
+			(effects
+				(font
+					(size 1.27 1.27)
+				)
+				(hide yes)
+			)
+		)
 		(pin "1"
 		)
@@
 			)
 		)
-		(property "Footprint" ""
+		(property "Footprint" "Package_DIP:DIP-14_W7.62mm"
 			(at 48.26 85.09 0)
 			(effects
@@
 			)
 		)
+		(property "Order Link" "https://www.digikey.com/en/products/detail/texas-instruments/SN74LS04N/277275"
+			(at 48.26 85.09 0)
+			(effects
+				(font
+					(size 1.27 1.27)
+				)
+				(hide yes)
+			)
+		)
 		(pin "3"
 		)
@@
 			)
 		)
-		(property "Footprint" ""
+		(property "Footprint" "Package_DIP:DIP-14_W7.62mm"
 			(at 45.72 226.06 0)
 			(effects
@@
 			)
 		)
+		(property "Order Link" "https://www.digikey.com/en/products/detail/texas-instruments/SN74LS04N/277275"
+			(at 45.72 226.06 0)
+			(effects
+				(font
+					(size 1.27 1.27)
+				)
+				(hide yes)
+			)
+		)
 		(pin "1"
 		)
@@
 	)
 	(symbol
-		(lib_id "sun2:74F74")
-		(at -33.02 180.34 0)
-		(unit 2)
-		(exclude_from_sim no)
-		(in_bom yes)
-		(on_board yes)
-		(dnp no)
-		(fields_autoplaced yes)
-		(property "Reference" "U206"
-			(at -30.8767 170.18 0)
-			(effects
-				(font
-					(size 1.27 1.27)
-				)
-				(justify left)
-			)
-		)
-		(property "Value" "74F74"
-			(at -30.8767 172.72 0)
-			(effects
-				(font
-					(size 1.27 1.27)
-				)
-				(justify left)
-			)
-		)
-		(property "Footprint" "Package_DIP:DIP-14_W7.62mm"
-			(at -33.02 180.34 0)
-			(effects
-				(font
-					(size 1.27 1.27)
-				)
-				(hide yes)
-			)
-		)
-		(property "Datasheet" "https://www.ti.com/lit/ds/symlink/sn74f74.pdf"
-			(at -33.02 180.34 0)
-			(effects
-				(font
-					(size 1.27 1.27)
-				)
-				(hide yes)
-			)
-		)
-		(property "Description" "Dual D Flip-flop, Set & Reset"
-			(at -33.02 180.34 0)
-			(effects
-				(font
-					(size 1.27 1.27)
-				)
-				(hide yes)
-			)
-		)
-		(property "Order Link" "https://www.digikey.com/en/products/detail/texas-instruments/SN74F74N/277204"
-			(at -33.02 180.34 0)
-			(effects
-				(font
-					(size 1.27 1.27)
-				)
-				(hide yes)
-			)
-		)
-		(pin "7"
-		)
-		(pin "14"
-		)
-		(pin "13"
-		)
-		(pin "10"
-		)
-		(pin "9"
-		)
-		(pin "8"
-		)
-		(pin "5"
-		)
-		(pin "1"
-		)
-		(pin "4"
-		)
-		(pin "3"
-		)
-		(pin "2"
-		)
-		(pin "12"
-		)
-		(pin "6"
-		)
-		(pin "11"
-		)
-		(instances
-			(project ""
-				(path "/67ee2072-0b57-4a50-8537-b17b5f651e89/2d3d381d-4c8b-4bfc-8adc-91fc2fe1e9d0"
-					(reference "U206")
-					(unit 2)
-				)
-			)
-		)
-	)
-	(symbol
 		(lib_id "sun2:74LS04")
 		(at -29.21 149.86 0)
@@
 			)
 		)
-		(property "Footprint" ""
+		(property "Footprint" "Package_DIP:DIP-14_W7.62mm"
 			(at -29.21 149.86 0)
 			(effects
@@
 			)
 		)
+		(property "Order Link" "https://www.digikey.com/en/products/detail/texas-instruments/SN74LS04N/277275"
+			(at -29.21 149.86 0)
+			(effects
+				(font
+					(size 1.27 1.27)
+				)
+				(hide yes)
+			)
+		)
 		(pin "3"
 		)
@@
 			)
 		)
-		(property "Footprint" ""
+		(property "Footprint" "Package_DIP:DIP-14_W7.62mm"
 			(at 92.71 173.99 0)
 			(effects
@@
 			)
 		)
+		(property "Order Link" "https://www.digikey.com/en/products/detail/texas-instruments/SN74LS04N/277275"
+			(at 92.71 173.99 0)
+			(effects
+				(font
+					(size 1.27 1.27)
+				)
+				(hide yes)
+			)
+		)
 		(pin "1"
 		)
@@
 			)
 		)
-		(property "Footprint" ""
+		(property "Footprint" "Package_DIP:DIP-14_W7.62mm"
 			(at 196.85 233.68 0)
 			(effects
@@
 			)
 		)
+		(property "Order Link" "https://www.digikey.com/en/products/detail/texas-instruments/SN74LS04N/277275"
+			(at 196.85 233.68 0)
+			(effects
+				(font
+					(size 1.27 1.27)
+				)
+				(hide yes)
+			)
+		)
 		(pin "3"
 		)
@@
 			)
 		)
-		(property "Footprint" ""
+		(property "Footprint" "Package_DIP:DIP-14_W7.62mm"
 			(at -29.21 140.97 0)
 			(effects
@@
 			)
 		)
+		(property "Order Link" "https://www.digikey.com/en/products/detail/texas-instruments/SN74LS04N/277275"
+			(at -29.21 140.97 0)
+			(effects
+				(font
+					(size 1.27 1.27)
+				)
+				(hide yes)
+			)
+		)
 		(pin "3"
 		)
@@
 			)
 		)
-		(property "Footprint" ""
+		(property "Footprint" "Package_DIP:DIP-14_W7.62mm"
 			(at 73.66 226.06 0)
 			(effects
@@
 			)
 		)
+		(property "Order Link" "https://www.digikey.com/en/products/detail/texas-instruments/SN74LS04N/277275"
+			(at 73.66 226.06 0)
+			(effects
+				(font
+					(size 1.27 1.27)
+				)
+				(hide yes)
+			)
+		)
 		(pin "1"
 		)
@@
 			)
 		)
-		(property "Footprint" ""
+		(property "Footprint" "Package_DIP:DIP-14_W7.62mm"
 			(at 102.87 226.06 0)
 			(effects
@@
 			(effects
 				(font
+					(size 1.27 1.27)
+				)
+				(hide yes)
+			)
+		)
+		(property "Order Link" "https://www.digikey.com/en/products/detail/texas-instruments/SN74LS04N/277275"
+			(at 102.87 226.06 0)
+			(effects
+				(font

Commit message: work on addresses and buffers
Parts:
- removed unit 3 of U102
Changed lines of the file:
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@@
-	)
-	(symbol
-		(lib_id "sun2:74F00")
-		(at -33.02 66.04 0)
-		(unit 3)
-		(exclude_from_sim no)
-		(in_bom yes)
-		(on_board yes)
-		(dnp no)
-		(property "Reference" "U102"
-			(at -33.274 64.77 0)
-			(effects
-				(font
-					(size 1.27 1.27)
-				)
-			)
-		)
-		(property "Value" "74F00"
-			(at -33.274 67.31 0)
-			(effects
-				(font
-					(size 1.27 1.27)
-				)
-			)
-		)
-		(property "Footprint" "Package_DIP:DIP-14_W7.62mm"
-			(at -33.02 66.04 0)
-			(effects
-				(font
-					(size 1.27 1.27)
-				)
-				(hide yes)
-			)
-		)
-		(property "Datasheet" "https://www.ti.com/lit/ds/symlink/sn74f00.pdf"
-			(at -33.02 66.04 0)
-			(effects
-				(font
-					(size 1.27 1.27)
-				)
-				(hide yes)
-			)
-		)
-		(property "Description" "quad 2-input NAND gate"
-			(at -33.02 66.04 0)
-			(effects
-				(font
-					(size 1.27 1.27)
-				)
-				(hide yes)
-			)
-		)
-		(property "Order Link" "https://www.digikey.com/en/products/detail/texas-instruments/SN74F00N/373665"
-			(at -33.02 66.04 0)
-			(effects
-				(font
-					(size 1.27 1.27)
-				)
-				(hide yes)
-			)
-		)
-		(pin "4"
-		)
-		(pin "9"
-		)
-		(pin "5"
-		)
-		(pin "6"
-		)
-		(pin "13"
-		)
-		(pin "11"
-		)
-		(pin "3"
-		)
-		(pin "1"
-		)
-		(pin "2"
-		)
-		(pin "12"
-		)
-		(pin "10"
-		)
-		(pin "8"
-		)
-		(pin "14"
-		)
-		(pin "7"
-		)
-		(instances
-			(project ""
-				(path "/67ee2072-0b57-4a50-8537-b17b5f651e89/2d3d381d-4c8b-4bfc-8adc-91fc2fe1e9d0"
-					(reference "U102")
-					(unit 3)
-				)
-			)
-		)
 	)
 	(symbol

Commit message: Dedup U608 and U610
Parts:
- removed unit 2 of U608
- removed unit 7 of U608
- removed unit 1 of U608
- removed unit 3 of U608
- removed unit 5 of U608
- removed unit 3 of U610
- removed unit 2 of U610
- removed unit 1 of U610
- removed unit 5 of U610
- removed unit 7 of U610
- removed unit 4 of U610
Other:
- moved on the sheet: U110D, U122C, U206C

Commit message: Finish connectors
Changed lines of the file:
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@@
 	)
 	(hierarchical_label "POR\\"
-		(shape input)
+		(shape output)
 		(at 57.15 44.45 180)
 		(effects

Commit message: Finish passives
Parts:
- removed unit 5 of U102
- removed unit 5 of U109
- removed unit 7 of U110
- removed unit 2 of U111
- removed unit 3 of U114
- removed unit 7 of U115
- removed unit 7 of U122
- removed unit 3 of U206
Connections:
- no-connect marks 0 -> 9
Other:
- moved on the sheet: U110D, U114B, U122C

Commit message: Start global connections, error fixes
Parts:
- removed unit 4 of U608
Connections:
- net P.BACK\: now also U206.4 (~{S})
- net P.RESET\: now also U110.9
- net P1.INIT\: now also U110.8
- no-connect marks 9 -> 8
Other:
- moved on the sheet: U110D
