File: schematics/kicad/sun2_passive.kicad_sch (KiCad schematic)
At the start: 78 parts, among them U101 74F32, U102 74F00, U109 74F08, U110 7407, U111 74F251, U114 74LS20, U115 74F04, U122 7406, U201 74F74, U203 74F74, U204 74F74, U205 74F74, U206 74F74, U207 74F74, U209 74LS393, U211 P20X10, U313 74F08, U422 74LS08, U503 74F32, U508 74F02, U512 74F74, U513 74F00, U520 74LS20, U608 74LS04, U610 74LS04, U613 74LS05, U703 74F08, U709 74F74, X1 0.1uF, X10 0.1uF, X11 0.1uF, X12 0.1uF, X13 0.1uF, X14 0.1uF, X15 0.1uF, X16 0.1uF, X17 0.1uF, X18 0.1uF, X19 0.1uF, X2 0.1uF, X20 0.1uF, X21 0.1uF, X22 0.1uF, X23 0.1uF, X24 0.1uF, X25 0.1uF, X26 0.1uF, X27 0.1uF, X28 0.1uF, X29 0.1uF, X3 0.1uF, X30 0.1uF, X31 0.1uF, X32 0.1uF, X33 0.1uF, X34 0.1uF, X35 0.1uF, X36 0.1uF, X37 0.1uF, X38 0.1uF, X39 0.1uF, X4 0.1uF, X40 0.1uF, X41 0.1uF, X42 0.1uF, X43 0.1uF, X44 0.1uF, X45 0.1uF, X46 0.1uF, X47 0.1uF, X48 0.1uF, X49 0.1uF, X5 0.1uF, X50 0.1uF, X6 0.1uF, X7 0.1uF, X8 0.1uF, X9 0.1uF

Commit message: Start global connections, error fixes
Changed lines of the file:
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@@
 	)
 	(junction
+		(at 101.6 45.72)
+		(diameter 0)
+		(color 0 0 0 0)
+	)
+	(junction
 		(at 118.11 151.13)
 		(diameter 0)
@@
 	)
 	(junction
+		(at 101.6 20.32)
+		(diameter 0)
+		(color 0 0 0 0)
+	)
+	(junction
 		(at 147.32 151.13)
 		(diameter 0)
@@
 	(wire
 		(pts
+			(xy 101.6 20.32) (xy 113.03 20.32)
+		)
+		(stroke
+			(width 0)
+			(type default)
+		)
+	)
+	(wire
+		(pts
 			(xy 161.29 91.44) (xy 171.45 91.44)
 		)
@@
 	(wire
 		(pts
+			(xy 101.6 45.72) (xy 113.03 45.72)
+		)
+		(stroke
+			(width 0)
+			(type default)
+		)
+	)
+	(wire
+		(pts
 			(xy 100.33 77.47) (xy 110.49 77.47)
 		)
@@
 	(wire
 		(pts
-			(xy 97.79 45.72) (xy 113.03 45.72)
+			(xy 97.79 45.72) (xy 101.6 45.72)
 		)
 		(stroke
@@
 	(wire
 		(pts
-			(xy 97.79 20.32) (xy 113.03 20.32)
+			(xy 97.79 20.32) (xy 101.6 20.32)
 		)
 		(stroke
@@
 	)
 	(symbol
+		(lib_id "power:GND")
+		(at 101.6 45.72 0)
+		(unit 1)
+		(exclude_from_sim no)
+		(in_bom yes)
+		(on_board yes)
+		(dnp no)
+		(fields_autoplaced yes)
+		(property "Reference" "#PWR039"
+			(at 101.6 52.07 0)
+			(effects
+				(font
+					(size 1.27 1.27)
+				)
+				(hide yes)
+			)
+		)
+		(property "Value" "GND"
+			(at 101.6 50.8 0)
+			(effects
+				(font
+					(size 1.27 1.27)
+				)
+			)
+		)
+		(property "Footprint" ""
+			(at 101.6 45.72 0)
+			(effects
+				(font
+					(size 1.27 1.27)
+				)
+				(hide yes)
+			)
+		)
+		(property "Datasheet" ""
+			(at 101.6 45.72 0)
+			(effects
+				(font
+					(size 1.27 1.27)
+				)
+				(hide yes)
+			)
+		)
+		(property "Description" "Power symbol creates a global label with name \"GND\" , ground"
+			(at 101.6 45.72 0)
+			(effects
+				(font
+					(size 1.27 1.27)
+				)
+				(hide yes)
+			)
+		)
+		(pin "1"
+		)
+		(instances
+			(project ""
+				(path "/67ee2072-0b57-4a50-8537-b17b5f651e89/8f1c8a72-97e7-46bf-a4c9-b87b7a1a1f7c"
+					(reference "#PWR039")
+					(unit 1)
+				)
+			)
+		)
+	)
+	(symbol
 		(lib_id "Device:C_Small")
 		(at 100.33 80.01 0)
@@
 				)
 			)
+		)
+	)
+	(symbol
+		(lib_id "power:VCC")
+		(at 101.6 20.32 0)
+		(unit 1)
+		(exclude_from_sim no)
+		(in_bom yes)
+		(on_board yes)
+		(dnp no)
+		(fields_autoplaced yes)
+		(property "Reference" "#PWR040"
+			(at 101.6 24.13 0)
+			(effects
+				(font
+					(size 1.27 1.27)
+				)
+				(hide yes)
+			)
+		)
+		(property "Value" "VCC"
+			(at 101.6 15.24 0)
+			(effects
+				(font
+					(size 1.27 1.27)
+				)
+			)
+		)
+		(property "Footprint" ""
+			(at 101.6 20.32 0)
+			(effects
+				(font
+					(size 1.27 1.27)
+				)
+				(hide yes)
+			)
+		)
+		(property "Datasheet" ""
+			(at 101.6 20.32 0)
+			(effects
+				(font
+					(size 1.27 1.27)
+				)
+				(hide yes)
+			)
+		)
+		(property "Description" "Power symbol creates a global label with name \"VCC\""
+			(at 101.6 20.32 0)
+			(effects
+				(font
+					(size 1.27 1.27)
+				)
+				(hide yes)
+			)
+		)
+		(pin "1"
+		)
+		(instances
+			(project ""
+				(path "/67ee2072-0b57-4a50-8537-b17b5f651e89/8f1c8a72-97e7-46bf-a4c9-b87b7a1a1f7c"
+					(reference "#PWR040")
+					(unit 1)
+				)
+			)
