File: schematics/kicad/sun2_prom_rtc_regs.kicad_sch (KiCad schematic)
At the start: 11 parts, among them U400 74F138, U401 74F138, U402 74F138, U406 27256, U407 27256, U411 74S288, U412 74LS534, U413 74LS273, U414 74LS244, U420 58167, U422 74LS08

Commit message: Finish PROM, RTC, Registers
Parts:
- added C400: 22pF+, symbol Device:C_Small
- added C401: 22pF, symbol Device:C_Small
- added K401: TODO, symbol Device:C_Polarized_Small
- added R400: 200k, symbol Device:R_Small_US
- added R401: 100, symbol Device:R_Small_US
- added R402: 10k, symbol Device:R_Small_US
- added U101: 74F32, Package_DIP:DIP-14_W7.62mm, symbol sun2:74F32
- added U421: 32768Hz, symbol Device:Crystal
- added U424: 3V, symbol Device:Battery_Cell
- added U425, U426, U427 (x3): 1N4148, Diode_THT:D_DO-35_SOD27_P7.62mm_Horizontal, symbol Diode:1N4148
Connections:
- net BOOT\: now also U101.12
- net GND: now also U406.20 (~{CE}), U407.20 (~{CE}), U420.1 (CS), U420.12 (GND), C400.1, C401.2, K401.2, R402.1, U424.2 (-)
- net P.A11: now also U406.21 (A10), U407.21 (A10)
- net P.A12: now also U406.23 (A11), U407.23 (A11)
- net P.A13: now also U406.2 (A12), U407.2 (A12)
- net P.A14: now also U406.26 (A13), U407.26 (A13)
- net P.A15: now also U406.27 (A14), U407.27 (A14)
- net P.D0: now also U406.11 (D0)
- net P.D1: now also U406.12 (D1)
- net P.D10: now also U407.13 (D2), U420.17 (D2)
- net P.D11: now also U407.15 (D3), U420.18 (D3)
- net P.D12: now also U407.16 (D4), U420.19 (D4)
- net P.D13: now also U407.17 (D5), U420.20 (D5)
- net P.D14: now also U407.18 (D6), U420.21 (D6)
- net P.D15: now also U407.19 (D7), U420.22 (D7)
- net P.D2: now also U406.13 (D2)
- net P.D3: now also U406.15 (D3)
- net P.D4: now also U406.16 (D4)
- net P.D5: now also U406.17 (D5)
- net P.D6: now also U406.18 (D6)
- net P.D7: now also U406.19 (D7)
- net P.D8: now also U407.11 (D0), U420.15 (D0)
- net P.D9: now also U407.12 (D1), U420.16 (D1)
- net VCC: now also U401.6 (E3), U402.6 (E3), U406.1 (VPP), U407.1 (VPP), U425.2 (A)
- net P.A1: now reaches U406.10 (A0)
- net P.A1: now also U407.10 (A0), U420.5 (A0)
- net at U406.22 (~{OE}): now also U407.22 (~{OE}), U422.11
- net P.A10: now reaches U406.24 (A9)
- net P.A10: now also U407.24 (A9)
- net P.A9: now reaches U406.25 (A8)
- net P.A9: now also U407.25 (A8)
- net P.A8: now reaches U406.3 (A7)
- net P.A8: now also U407.3 (A7)
- net P.A7: now reaches U406.4 (A6)
- net P.A7: now also U407.4 (A6)
- net P.A6: now reaches U406.5 (A5)
- net P.A6: now also U407.5 (A5)
- net P.A5: now reaches U406.6 (A4)
- net P.A5: now also U407.6 (A4), U420.9 (A4)
- net P.A4: now reaches U406.7 (A3)
- net P.A4: now also U407.7 (A3), U420.8 (A3)
- net P.A3: now reaches U406.8 (A2)
- net P.A3: now also U407.8 (A2), U420.7 (A2)
- net P.A2: now reaches U406.9 (A1)
- net P.A2: now also U407.9 (A1), U420.6 (A1)
- net TYPE0: now reaches U400.1 (A0)
- net WR.IO\: now reaches U400.10 (O5)
- net WR.IO\: now also U402.5 (E2)
- net WR.RAM\: now reaches U400.11 (O4)
- net IORC\: now reaches U400.12 (O3)
- net MRDC\: now reaches U400.13 (O2)
- net RD.IO\: now reaches U400.14 (O1)
- net RD.IO\: now also U401.5 (E2)
- net RD.RAM\: now reaches U400.15 (O0)
- net TYPE1: now reaches U400.2 (A1)
- net R\/W: now reaches U400.3 (A2)
- net ERR: now reaches U400.4 (E1)
- net DS\: now reaches U400.5 (E2)
- net C.S5: now reaches U400.6 (E3)
- net IOWC\: now reaches U400.7 (O7)
- net MWTC\: now reaches U400.9 (O6)
- net MA11: now reaches U401.1 (A0)
- net MA11: now also U402.1 (A0)
- net RD.TIMER\: now reaches U401.10 (O5)
- net RD.SCC\: now reaches U401.11 (O4)
- net RD.PORT\: now reaches U401.12 (O3)
- net RD.DCP\: now reaches U401.13 (O2)
- net RD.FPP\: now reaches U401.14 (O1)
- net RD.PROM\: now reaches U401.15 (O0)
- net RD.PROM\: now also U422.12
- net MA12: now reaches U401.2 (A1)
- net MA12: now also U402.2 (A1)
- net MA13: now reaches U401.3 (A2)
- net MA13: now also U402.3 (A2)
- net MA14: now reaches U401.4 (E1)
- net MA14: now also U402.4 (E1)
- net RD.RTC\: now reaches U401.7 (O7)
- net RD.RTC\: now also U420.2 (RD), U422.1
- net RD.ROP\: now reaches U401.9 (O6)
- net WR.TIMER\: now reaches U402.10 (O5)
- net WR.SCC\: now reaches U402.11 (O4)
- net WR.DCP\: now reaches U402.13 (O2)
- net WR.FPP\: now reaches U402.14 (O1)
- net WR.RTC\: now reaches U402.7 (O7)
- net WR.RTC\: now also U420.3 (WR), U422.2
- net WR.ROP\: now reaches U402.9 (O6)
- net at U420.10 (XI): now also C400.2, U421.1
- net at U420.11 (XO): now also R400.2
- net at U420.23 (PD): now also R402.2, U427.1 (K)
- net at U420.24 (VCC): now also K401.1, U425.1 (K), U426.1 (K)
- net at U422.3: now also U422.4
- net P.INTA\: now reaches U422.5
- net P.VPA\: now reaches U422.6
- net BOOTEN\: now reaches U422.13
- net BOOTEN\: now also U101.11
- new net: R401.2, U426.2 (A)
- new net: U427.1 (K), U427.2 (A) (x2)
- new net: R401.1, U424.1 (+)
- new net: C401.1, R400.1, U421.2
- new net P.SPROG\: U101.13
- new net POR\: U427.2 (A)
- no-connect marks 0 -> 5
Other:
- note added: "BOOT PROMS"
- note added: "BUS ERROR REG."
- note added: "ID PROM"
- note added: "REAL-TIME CLOCK"
- note added: "STROBE DECODERS"
- note added: "SYSTEM ENABLE REG."
- moved on the sheet: U407, U420, U422A, U422B, U422D

Commit message: Start on rasterop, parity, P2
Parts:
- removed unit 3 of U101
- removed unit 3 of U422
Changed lines of the file:
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@@
-	)
-	(symbol
-		(lib_id "74xx:74LS08")
-		(at -13.97 106.68 0)
-		(unit 3)
-		(exclude_from_sim no)
-		(in_bom yes)
-		(on_board yes)
-		(dnp no)
-		(fields_autoplaced yes)
-		(property "Reference" "U422"
-			(at -13.9783 97.79 0)
-			(effects
-				(font
-					(size 1.27 1.27)
-				)
-			)
-		)
-		(property "Value" "74LS08"
-			(at -13.9783 100.33 0)
-			(effects
-				(font
-					(size 1.27 1.27)
-				)
-			)
-		)
-		(property "Footprint" "Package_DIP:DIP-14_W7.62mm"
-			(at -13.97 106.68 0)
-			(effects
-				(font
-					(size 1.27 1.27)
-				)
-				(hide yes)
-			)
-		)
-		(property "Datasheet" "http://www.ti.com/lit/gpn/sn74LS08"
-			(at -13.97 106.68 0)
-			(effects
-				(font
-					(size 1.27 1.27)
-				)
-				(hide yes)
-			)
-		)
-		(property "Description" "Quad And2"
-			(at -13.97 106.68 0)
-			(effects
-				(font
-					(size 1.27 1.27)
-				)
-				(hide yes)
-			)
-		)
-		(property "Order Link" "https://www.digikey.com/en/products/detail/texas-instruments/SN74LS08N/277279"
-			(at -13.97 106.68 0)
-			(effects
-				(font
-					(size 1.27 1.27)
-				)
-				(hide yes)
-			)
-		)
-		(pin "9"
-		)
-		(pin "8"
-		)
-		(pin "10"
-		)
-		(pin "14"
-		)
-		(pin "11"
-		)
-		(pin "13"
-		)
-		(pin "7"
-		)
-		(pin "12"
-		)
-		(pin "6"
-		)
-		(pin "3"
-		)
-		(pin "2"
-		)
-		(pin "5"
-		)
-		(pin "1"
-		)
-		(pin "4"
-		)
-		(instances
-			(project ""
-				(path "/67ee2072-0b57-4a50-8537-b17b5f651e89/b42ede88-616c-473e-8f95-b5ba6ef10988"
-					(reference "U422")
-					(unit 3)
-				)
-			)
-		)
 	)
 	(symbol
@@
 				)
 			)
-		)
-	)
-	(symbol
-		(lib_id "sun2:74F32")
-		(at -39.37 135.89 0)
-		(unit 3)
-		(exclude_from_sim no)
-		(in_bom yes)
-		(on_board yes)
-		(dnp no)
-		(fields_autoplaced yes)
-		(property "Reference" "U101"
-			(at -39.37 127 0)
-			(effects
-				(font
-					(size 1.27 1.27)
-				)
-			)
-		)
-		(property "Value" "74F32"
-			(at -39.37 129.54 0)
-			(effects
-				(font
-					(size 1.27 1.27)
-				)
-			)
-		)
-		(property "Footprint" "Package_DIP:DIP-14_W7.62mm"
-			(at -39.37 135.89 0)
-			(effects
-				(font
-					(size 1.27 1.27)
-				)
-				(hide yes)
-			)
-		)
-		(property "Datasheet" "https://www.ti.com/lit/ds/symlink/sn74f32.pdf"
-			(at -39.37 135.89 0)
-			(effects
-				(font
-					(size 1.27 1.27)
-				)
-				(hide yes)
-			)
-		)
-		(property "Description" "Quad 2-input OR"
-			(at -39.37 135.89 0)
-			(effects
-				(font
-					(size 1.27 1.27)
-				)
-				(hide yes)
-			)
-		)
-		(property "Order Link" "https://www.digikey.com/en/products/detail/texas-instruments/SN74F32N/373722"
-			(at -39.37 135.89 0)
-			(effects
-				(font
-					(size 1.27 1.27)
-				)
-				(hide yes)
-			)
-		)
-		(pin "2"
-		)
-		(pin "3"
-		)
-		(pin "6"
-		)
-		(pin "1"
-		)
-		(pin "5"
-		)
-		(pin "4"
-		)
-		(pin "7"
-		)
-		(pin "8"
-		)
-		(pin "10"
-		)
-		(pin "12"
-		)
-		(pin "13"
-		)
-		(pin "11"
-		)
-		(pin "9"
-		)
-		(pin "14"
-		)
-		(instances
-			(project ""
-				(path "/67ee2072-0b57-4a50-8537-b17b5f651e89/b42ede88-616c-473e-8f95-b5ba6ef10988"
-					(reference "U101")
-					(unit 3)
-				)
-			)

Commit message: work on addresses and buffers
Parts:
- removed unit 1 of U101
Changed lines of the file:
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@@
-	)
-	(symbol
-		(lib_id "sun2:74F32")
-		(at -55.88 119.38 0)
-		(unit 1)
-		(exclude_from_sim no)
-		(in_bom yes)
-		(on_board yes)
-		(dnp no)
-		(fields_autoplaced yes)
-		(property "Reference" "U101"
-			(at -55.88 110.49 0)
-			(effects
-				(font
-					(size 1.27 1.27)
-				)
-			)
-		)
-		(property "Value" "74F32"
-			(at -55.88 113.03 0)
-			(effects
-				(font
-					(size 1.27 1.27)
-				)
-			)
-		)
-		(property "Footprint" "Package_DIP:DIP-14_W7.62mm"
-			(at -55.88 119.38 0)
-			(effects
-				(font
-					(size 1.27 1.27)
-				)
-				(hide yes)
-			)
-		)
-		(property "Datasheet" "https://www.ti.com/lit/ds/symlink/sn74f32.pdf"
-			(at -55.88 119.38 0)
-			(effects
-				(font
-					(size 1.27 1.27)
-				)
-				(hide yes)
-			)
-		)
-		(property "Description" "Quad 2-input OR"
-			(at -55.88 119.38 0)
-			(effects
-				(font
-					(size 1.27 1.27)
-				)
-				(hide yes)
-			)
-		)
-		(property "Order Link" "https://www.digikey.com/en/products/detail/texas-instruments/SN74F32N/373722"
-			(at -55.88 119.38 0)
-			(effects
-				(font
-					(size 1.27 1.27)
-				)
-				(hide yes)
-			)
-		)
-		(pin "2"
-		)
-		(pin "3"
-		)
-		(pin "6"
-		)
-		(pin "1"
-		)
-		(pin "5"
-		)
-		(pin "4"
-		)
-		(pin "7"
-		)
-		(pin "8"
-		)
-		(pin "10"
-		)
-		(pin "12"
-		)
-		(pin "13"
-		)
-		(pin "11"
-		)
-		(pin "9"
-		)
-		(pin "14"
-		)
-		(instances
-			(project ""
-				(path "/67ee2072-0b57-4a50-8537-b17b5f651e89/b42ede88-616c-473e-8f95-b5ba6ef10988"
-					(reference "U101")
-					(unit 1)
-				)
-			)
-		)
 	)
 	(symbol

Commit message: Finish passives
Parts:
- removed unit 5 of U101
- removed unit 5 of U422
Connections:
- no-connect marks 5 -> 8
Other:
- moved on the sheet: U101B
Changed lines of the file:
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@@
 	)
 	(no_connect
+		(at 185.42 157.48)
+	)
+	(no_connect
 		(at 50.8 115.57)
 	)
@@
 		(at 238.76 93.98)
 	)
+	(no_connect
+		(at 200.66 160.02)
+	)
+	(no_connect
+		(at 185.42 162.56)
+	)
 	(bus_entry
 		(at 127 57.15)
@@
 	(symbol
 		(lib_id "sun2:74F32")
-		(at -57.15 134.62 0)
+		(at 193.04 160.02 0)
 		(unit 2)
 		(exclude_from_sim no)
@@
 		(fields_autoplaced yes)
 		(property "Reference" "U101"
-			(at -57.15 125.73 0)
+			(at 193.04 151.13 0)
 			(effects
 				(font
@@
 		)
 		(property "Value" "74F32"
-			(at -57.15 128.27 0)
+			(at 193.04 153.67 0)
 			(effects
 				(font
@@
 		)
 		(property "Footprint" "Package_DIP:DIP-14_W7.62mm"
-			(at -57.15 134.62 0)
+			(at 193.04 160.02 0)
 			(effects
 				(font
@@
 		)
 		(property "Datasheet" "https://www.ti.com/lit/ds/symlink/sn74f32.pdf"
-			(at -57.15 134.62 0)
+			(at 193.04 160.02 0)
 			(effects
 				(font
@@
 		)
 		(property "Description" "Quad 2-input OR"
-			(at -57.15 134.62 0)
+			(at 193.04 160.02 0)
 			(effects
 				(font
@@
 		)
 		(property "Order Link" "https://www.digikey.com/en/products/detail/texas-instruments/SN74F32N/373722"
-			(at -57.15 134.62 0)
+			(at 193.04 160.02 0)
 			(effects
 				(font
@@
 	)
 	(symbol
-		(lib_id "74xx:74LS08")
-		(at -15.24 133.35 0)
-		(unit 5)
-		(exclude_from_sim no)
-		(in_bom yes)
-		(on_board yes)
-		(dnp no)
-		(fields_autoplaced yes)
-		(property "Reference" "U422"
-			(at -7.62 132.0799 0)
-			(effects
-				(font
-					(size 1.27 1.27)
-				)
-				(justify left)
-			)
-		)
-		(property "Value" "74LS08"
-			(at -7.62 134.6199 0)
-			(effects
-				(font
-					(size 1.27 1.27)
-				)
-				(justify left)
-			)
-		)
-		(property "Footprint" "Package_DIP:DIP-14_W7.62mm"
-			(at -15.24 133.35 0)
-			(effects
-				(font
-					(size 1.27 1.27)
-				)
-				(hide yes)
-			)
-		)
-		(property "Datasheet" "http://www.ti.com/lit/gpn/sn74LS08"
-			(at -15.24 133.35 0)
-			(effects
-				(font
-					(size 1.27 1.27)
-				)
-				(hide yes)
-			)
-		)
-		(property "Description" "Quad And2"
-			(at -15.24 133.35 0)
-			(effects
-				(font
-					(size 1.27 1.27)
-				)
-				(hide yes)
-			)
-		)
-		(property "Order Link" "https://www.digikey.com/en/products/detail/texas-instruments/SN74LS08N/277279"
-			(at -15.24 133.35 0)
-			(effects
-				(font
-					(size 1.27 1.27)
-				)
-				(hide yes)
-			)
-		)
-		(pin "9"
-		)
-		(pin "8"
-		)
-		(pin "10"
-		)
-		(pin "14"
-		)
-		(pin "11"
-		)
-		(pin "13"
-		)
-		(pin "7"
-		)
-		(pin "12"
-		)
-		(pin "6"
-		)
-		(pin "3"
-		)
-		(pin "2"
-		)
-		(pin "5"
-		)
-		(pin "1"
-		)
-		(pin "4"
-		)
-		(instances
-			(project ""
-				(path "/67ee2072-0b57-4a50-8537-b17b5f651e89/b42ede88-616c-473e-8f95-b5ba6ef10988"
-					(reference "U422")
-					(unit 5)
-				)
-			)
-		)
-	)
-	(symbol
 		(lib_id "power:GND")
 		(at 241.3 156.21 0)
@@
 				)
 			)
-		)
-	)
-	(symbol
-		(lib_id "sun2:74F32")
-		(at -76.2 130.81 0)
-		(unit 5)
-		(exclude_from_sim no)
-		(in_bom yes)
-		(on_board yes)
-		(dnp no)
-		(fields_autoplaced yes)
-		(property "Reference" "U101"
-			(at -69.85 129.5399 0)
-			(effects
-				(font
-					(size 1.27 1.27)
-				)
-				(justify left)
-			)
-		)
-		(property "Value" "74F32"
-			(at -69.85 132.0799 0)
-			(effects
-				(font
-					(size 1.27 1.27)
-				)
-				(justify left)
-			)
-		)
-		(property "Footprint" "Package_DIP:DIP-14_W7.62mm"
-			(at -76.2 130.81 0)
-			(effects
-				(font
-					(size 1.27 1.27)
-				)
-				(hide yes)
-			)
-		)
-		(property "Datasheet" "https://www.ti.com/lit/ds/symlink/sn74f32.pdf"
-			(at -76.2 130.81 0)
-			(effects
-				(font
-					(size 1.27 1.27)
-				)
-				(hide yes)
-			)
-		)
-		(property "Description" "Quad 2-input OR"
-			(at -76.2 130.81 0)
-			(effects
-				(font
-					(size 1.27 1.27)
-				)
-				(hide yes)
-			)
-		)
-		(property "Order Link" "https://www.digikey.com/en/products/detail/texas-instruments/SN74F32N/373722"
-			(at -76.2 130.81 0)
-			(effects
-				(font
-					(size 1.27 1.27)
-				)
-				(hide yes)
-			)
-		)
-		(pin "2"
-		)
-		(pin "3"
-		)
-		(pin "6"
-		)
-		(pin "1"
-		)
-		(pin "5"
-		)
-		(pin "4"
-		)
-		(pin "7"
-		)
-		(pin "8"
-		)
-		(pin "10"
-		)
-		(pin "12"
-		)
-		(pin "13"
-		)
-		(pin "11"
-		)
-		(pin "9"
-		)
-		(pin "14"
-		)
-		(instances
-			(project ""
-				(path "/67ee2072-0b57-4a50-8537-b17b5f651e89/b42ede88-616c-473e-8f95-b5ba6ef10988"
-					(reference "U101")
-					(unit 5)
-				)
-			)

Commit message: Start global connections, error fixes
Parts:
- renumbered U427 to U428, U427 to U429
